Commit message: Robot Base complete

File: src/main_package/description/inertial_macros.xacro (robot description, xacro)
@@ -11,4 +11,5 @@
                 ixx="${(1/12) * mass * (3*radius*radius + length*length)}"
                 ixy="0.0"
+                ixz="0.0"
                 iyy="${(1/12) * mass * (3*radius*radius + length*length)}"
                 iyz="0.0"

File: src/main_package/description/robot_core.xacro (robot description, xacro)
@@ -5,31 +5,57 @@
     <xacro:include filename="materials.xacro" />
     <!-- ROBOT PROPERTIES -->
-    <xacro:property name="chassis_length" value="0.5" />
-    <xacro:property name="chassis_width" value="0.5" />
-    <xacro:property name="chassis_height" value="0.5" />
+    <xacro:property name="metal_thickness" value="0.003" />
+    <xacro:property name="metal_density" value="7850.0" />
+    <!--
+    mass = width * height * metal_thickness * metal_density
+    mass = length * height * metal_thickness * metal_density
+    -->
+    <!-- CHASSIS & FRAME PROPS -->
+    <xacro:property name="chassis_length" value="0.500" />
+    <xacro:property name="chassis_width" value="0.500" />
+    <xacro:property name="chassis_inner_length" value="0.272" />
+    <xacro:property name="chassis_inner_width" value="0.272" />
+    <xacro:property name="chassis_outer_side" value="0.272" />
+    <xacro:property name="chassis_outer_corner" value="0.162" />
+    <xacro:property name="chassis_outer_thickness" value="0.020" />
+    <xacro:property name="chassis_height" value="0.120" />
+    <xacro:property name="chassis_clearance" value="0.030" />
+    <xacro:property name="chassis_empty_space_length" value="${(chassis_length - chassis_outer_thickness*4)/3}" />
+    <xacro:property name="chassis_empty_space_width" value="${(chassis_width - chassis_outer_thickness*4)/3}" />
+    <!-- WHEEL PROPS -->
+    <xacro:property name="wheel_radius" value="0.050" />
+    <xacro:property name="wheel_thickness" value="0.038" />
     <!-- BASE LINK -->
     <link name="base_link"></link>
+    <!-- CENTER LINK -->
+    <joint name="center_joint" type="fixed">
+        <parent link="base_link" />
+        <child link="center_link" />
+        <origin xyz="${chassis_inner_length/2} 0 0" />
+    </joint>
+    <link name="center_link"></link>
     <!-- CHASSIS LINK -->
     <joint name="chassis_joint" type="fixed">
         <parent link="base_link" />
         <child link="chassis" />
-        <origin xyz="0 0 0" />
+        <origin xyz="${chassis_inner_length/2} 0 0" />
     </joint>
     <link name="chassis">
         <visual>
-            <origin xyz="${chassis_length/2} 0 ${chassis_height/2}" />
-            <geometry>
-                <box size="${chassis_length} ${chassis_width} ${chassis_height}" />
-            </geometry>
-            <material name="white" />
-        </visual>
-        <collision>
-            <origin xyz="${chassis_length/2} 0 ${chassis_height/2}" />
-            <geometry>
-                <box size="{chassis_length} ${chassis_width} ${chassis_height}" />
-            </geometry>
-        </collision>
-        <xacro:inertial_box mass="1.0" x="${chassis_length}" y="${chassis_width}" z="${chassis_height}">
-            <origin xyz="${chassis_length/2} 0 ${chassis_height/2}" rpy="0 0 0" />
+            <origin xyz="0 0 ${chassis_height/2 + chassis_clearance}" />
+            <geometry>
+                <box size="${chassis_inner_length} ${chassis_inner_width} ${chassis_height}" />
+            </geometry>
+            <material name="white" />
+        </visual>
+        <collision>
+            <origin xyz="0 0 ${chassis_height/2 + chassis_clearance}" />
+            <geometry>
+                <box size="${chassis_inner_length} ${chassis_inner_width} ${chassis_height}" />
+            </geometry>
+        </collision>
+        <xacro:inertial_box mass="${chassis_inner_width * chassis_inner_length * metal_thickness * metal_density}"
+            x="${chassis_inner_length}" y="${chassis_inner_width}" z="${chassis_height}">
+            <origin xyz="0 0 ${chassis_height/2 + chassis_clearance}" rpy="0 0 0" />
         </xacro:inertial_box>
     </link>
@@ -37,3 +63,593 @@
         <material>Gazebo/White</material>
     </gazebo>
+    <!-- WHEELS -->
+    <!-- left wheel -->
+    <joint name="left_wheel_joint" type="continuous">
+        <parent link="chassis" />
+        <child link="left_wheel" />
+        <origin
+            xyz="-${chassis_inner_length/2 + wheel_thickness/2} ${chassis_inner_width/2 + wheel_thickness/2} ${wheel_radius/2}"
+            rpy="-${pi/2} 0 0.785" />
+        <axis xyz="0 0 -1" />
+    </joint>
+    <link name="left_wheel">
+        <visual>
+            <geometry>
+                <cylinder radius="${wheel_radius}" length="${wheel_thickness}" />
+            </geometry>
+            <material name="blue" />
+        </visual>
+        <collision>
+            <geometry>
+                <sphere radius="${wheel_radius}" />
+            </geometry>
+        </collision>{pi/2} <xacro:inertial_cylinder
+            mass="1.0" length="${wheel_thickness}" radius="${wheel_radius}">
+            <origin xyz="0 0 0" rpy="0 0 0" />
+        </xacro:inertial_cylinder>
+    </link>
+    <gazebo reference="left_wheel">
+        <material>Gazebo/Blue</material>
+    </gazebo>
+    <!-- front wheel -->
+    <joint name="front_wheel_joint" type="continuous">
+        <parent link="chassis" />
+        <child link="front_wheel" />
+        <origin
+            xyz="${chassis_inner_length/2 + wheel_thickness/2} ${chassis_inner_width/2 + wheel_thickness/2} ${wheel_radius/2}"
+            rpy="-${pi/2} 0 -0.785" />
+        <axis xyz="0 0 -1" />
+    </joint>
+    <link name="front_wheel">
+        <visual>
+            <geometry>
+                <cylinder radius="${wheel_radius}" length="${wheel_thickness}" />
+            </geometry>
+            <material name="red" />
+        </visual>
+        <collision>
+            <geometry>
+                <sphere radius="${wheel_radius}" />
+            </geometry>
+        </collision>
+        <xacro:inertial_cylinder mass="1.0" length="${wheel_thickness}" radius="${wheel_radius}">
+            <origin xyz="0 0 0" rpy="0 0 0" />
+        </xacro:inertial_cylinder>
+    </link>
+    <gazebo reference="front_wheel">
+        <material>Gazebo/Red</material>
+    </gazebo>
+    <!-- right wheel -->
+    <joint name="right_wheel_joint" type="continuous">
+        <parent link="chassis" />
+        <child link="right_wheel" />
+        <origin
+            xyz="${chassis_inner_length/2 + wheel_thickness/2} -${chassis_inner_width/2 + wheel_thickness/2} ${wheel_radius/2}"
+            rpy="${pi/2} ${pi} 0.785" />
+        <axis xyz="0 0 -1" />
+    </joint>
+    <link name="right_wheel">
+        <visual>
+            <geometry>
+                <cylinder radius="${wheel_radius}" length="${wheel_thickness}" />
+            </geometry>
+            <material name="blue" />
+        </visual>
+        <collision>
+            <geometry>
+                <sphere radius="${wheel_radius}" />
+            </geometry>
+        </collision>
+        <xacro:inertial_cylinder mass="1.0" length="${wheel_thickness}" radius="${wheel_radius}">
+            <origin xyz="0 0 0" rpy="0 0 0" />
+        </xacro:inertial_cylinder>
+    </link>
+    <gazebo reference="right_wheel">
+        <material>Gazebo/Blue</material>
+    </gazebo>
+    <!-- back wheel -->
+    <joint name="back_wheel_joint" type="continuous">
+        <parent link="chassis" />
+        <child link="back_wheel" />
+        <origin
+            xyz="-${chassis_inner_length/2 + wheel_thickness/2} -${chassis_inner_width/2 + wheel_thickness/2} ${wheel_radius/2}"
+            rpy="${pi/2} ${pi} -0.785" />
+        <axis xyz="0 0 -1" />
+    </joint>
+    <link name="back_wheel">
+        <visual>
+            <geometry>
+                <cylinder radius="${wheel_radius}" length="${wheel_thickness}" />
+            </geometry>
+            <material name="blue" />
+        </visual>
+        <collision>
+            <geometry>
+                <sphere radius="${wheel_radius}" />
+            </geometry>
+        </collision>
+        <xacro:inertial_cylinder mass="1.0" length="${wheel_thickness}" radius="${wheel_radius}">
+            <origin xyz="0 0 0" rpy="0 0 0" />
+        </xacro:inertial_cylinder>
+    </link>
+    <gazebo reference="back_wheel">
+        <material>Gazebo/Blue</material>
+    </gazebo>
+    <!--
+        FRAME
+    -->
+    <!-- CORNERS -->
+    <!-- left corner -->
+    <joint name="frame_left_corner_top_joint" type="fixed">
+        <parent link="center_link" />
+        <child link="frame_left_corner_top" />
+        <origin
+            xyz="-${chassis_length/2 - chassis_empty_space_length/2 + chassis_outer_thickness*135/360} ${chassis_width/2 - chassis_empty_space_width/2 + chassis_outer_thickness*135/360} ${chassis_height + chassis_clearance - chassis_outer_thickness/2}"
+            rpy="0 0 0.785" />
+    </joint>
+    <link name="frame_left_corner_top">
+        <visual>
+            <geometry>
+                <box size="${chassis_outer_corner} ${chassis_outer_thickness} ${chassis_outer_thickness}" />
+            </geometry>
+            <material name="white" />
+        </visual>
+        <collision>
+            <geometry>
+                <box size="${chassis_outer_corner} ${chassis_outer_thickness} ${chassis_outer_thickness}" />
+            </geometry>
+        </collision>
+        <xacro:inertial_box
+            mass="${chassis_outer_corner * chassis_outer_thickness * metal_thickness * 4 * metal_density}"
+            x="${chassis_outer_corner}" y="${chassis_outer_thickness}"
+            z="${chassis_outer_thickness}">
+            <origin xyz="0 0 0" rpy="0 0 0" />
+        </xacro:inertial_box>
+    </link>
+    <gazebo reference="frame_left_corner_top">
+        <material>Gazebo/White</material>
+    </gazebo>
+    <joint name="frame_left_corner_bottom_joint" type="fixed">
+        <parent link="center_link" />
+        <child link="frame_left_corner_bottom" />
+        <origin
+            xyz="-${chassis_length/2 - chassis_empty_space_length/2 + chassis_outer_thickness*135/360} ${chassis_width/2 - chassis_empty_space_width/2 + chassis_outer_thickness*135/360} ${chassis_clearance + chassis_outer_thickness/2}"
+            rpy="0 0 0.785" />
+    </joint>
+    <link name="frame_left_corner_bottom">
+        <visual>
+            <geometry>
+                <box size="${chassis_outer_corner} ${chassis_outer_thickness} ${chassis_outer_thickness}" />
+            </geometry>
+            <material name="white" />
+        </visual>
+        <collision>
+            <geometry>
+                <box size="${chassis_outer_corner} ${chassis_outer_thickness} ${chassis_outer_thickness}" />
+            </geometry>
+        </collision>
+        <xacro:inertial_box
+            mass="${chassis_outer_corner * chassis_outer_thickness * metal_thickness * 4 * metal_density}"
+            x="${chassis_outer_corner}" y="${chassis_outer_thickness}"
+            z="${chassis_outer_thickness}">
+            <origin xyz="0 0 0" rpy="0 0 0" />
+        </xacro:inertial_box>
+    </link>
+    <gazebo reference="frame_left_corner_bottom">
+        <material>Gazebo/White</material>
+    </gazebo>
+    <!-- front corner -->
+    <joint name="frame_front_corner_top_joint" type="fixed">
+        <parent link="center_link" />
+        <child link="frame_front_corner_top" />
+        <origin
+            xyz="${chassis_length/2 - chassis_empty_space_length/2 + chassis_outer_thickness*135/360} ${chassis_width/2 - chassis_empty_space_width/2 + chassis_outer_thickness*135/360} ${chassis_height + chassis_clearance - chassis_outer_thickness/2}"
+            rpy="0 0 -0.785" />
+    </joint>
+    <link name="frame_front_corner_top">
+        <visual>
+            <geometry>
+                <box size="${chassis_outer_corner} ${chassis_outer_thickness} ${chassis_outer_thickness}" />
+            </geometry>
+            <material name="white" />
+        </visual>
+        <collision>
+            <geometry>
+                <box size="${chassis_outer_corner} ${chassis_outer_thickness} ${chassis_outer_thickness}" />
+            </geometry>
+        </collision>
+        <xacro:inertial_box
+            mass="${chassis_outer_corner * chassis_outer_thickness * metal_thickness * 4 * metal_density}"
+            x="${chassis_outer_corner}" y="${chassis_outer_thickness}"
+            z="${chassis_outer_thickness}">
+            <origin xyz="0 0 0" rpy="0 0 0" />
+        </xacro:inertial_box>
+    </link>
+    <gazebo reference="frame_front_corner_top">
+        <material>Gazebo/White</material>
+    </gazebo>
+    <joint name="frame_front_corner_bottom_joint" type="fixed">
+        <parent link="center_link" />
+        <child link="frame_front_corner_bottom" />
+        <origin
+            xyz="${chassis_length/2 - chassis_empty_space_length/2 + chassis_outer_thickness*135/360} ${chassis_width/2 - chassis_empty_space_width/2 + chassis_outer_thickness*135/360} ${chassis_clearance + chassis_outer_thickness/2}"
+            rpy="0 0 -0.785" />
+    </joint>
+    <link name="frame_front_corner_bottom">
+        <visual>
+            <geometry>
+                <box size="${chassis_outer_corner} ${chassis_outer_thickness} ${chassis_outer_thickness}" />
+            </geometry>
+            <material name="white" />
+        </visual>
+        <collision>
+            <geometry>
+                <box size="${chassis_outer_corner} ${chassis_outer_thickness} ${chassis_outer_thickness}" />
+            </geometry>
+        </collision>
+        <xacro:inertial_box
+            mass="${chassis_outer_corner * chassis_outer_thickness * metal_thickness * 4 * metal_density}"
+            x="${chassis_outer_corner}" y="${chassis_outer_thickness}"
+            z="${chassis_outer_thickness}">
+            <origin xyz="0 0 0" rpy="0 0 0" />
+        </xacro:inertial_box>
+    </link>
+    <gazebo reference="frame_front_corner_bottom">
+        <material>Gazebo/White</material>
+    </gazebo>
+    <!-- right corner -->
+    <joint name="frame_right_corner_top_joint" type="fixed">
+        <parent link="center_link" />
+        <child link="frame_right_corner_top" />
+        <origin
+            xyz="${chassis_length/2 - chassis_empty_space_length/2 + chassis_outer_thickness*135/360} -${chassis_width/2 - chassis_empty_space_width/2 + chassis_outer_thickness*135/360} ${chassis_height + chassis_clearance - chassis_outer_thickness/2}"
+            rpy="0 0 0.785" />
+    </joint>
+    <link name="frame_right_corner_top">
+        <visual>
+            <geometry>
+                <box size="${chassis_outer_corner} ${chassis_outer_thickness} ${chassis_outer_thickness}" />
+            </geometry>
+            <material name="white" />
+        </visual>
+        <collision>
+            <geometry>
+                <box size="${chassis_outer_corner} ${chassis_outer_thickness} ${chassis_outer_thickness}" />
+            </geometry>
+        </collision>
+        <xacro:inertial_box
+            mass="${chassis_outer_corner * chassis_outer_thickness * metal_thickness * 4 * metal_density}"
+            x="${chassis_outer_corner}" y="${chassis_outer_thickness}"
+            z="${chassis_outer_thickness}">
+            <origin xyz="0 0 0" rpy="0 0 0" />
+        </xacro:inertial_box>
+    </link>
+    <gazebo reference="frame_right_corner_top">
+        <material>Gazebo/White</material>
+    </gazebo>
+    <joint name="frame_right_corner_bottom_joint" type="fixed">
+        <parent link="center_link" />
+        <child link="frame_right_corner_bottom" />
+        <origin
+            xyz="${chassis_length/2 - chassis_empty_space_length/2 + chassis_outer_thickness*135/360} -${chassis_width/2 - chassis_empty_space_width/2 + chassis_outer_thickness*135/360} ${chassis_clearance + chassis_outer_thickness/2}"
+            rpy="0 0 0.785" />
+    </joint>
+    <link name="frame_right_corner_bottom">
+        <visual>
+            <geometry>
+                <box size="${chassis_outer_corner} ${chassis_outer_thickness} ${chassis_outer_thickness}" />
+            </geometry>
+            <material name="white" />
+        </visual>
+        <collision>
+            <geometry>
+                <box size="${chassis_outer_corner} ${chassis_outer_thickness} ${chassis_outer_thickness}" />
+            </geometry>
+        </collision>
+        <xacro:inertial_box
+            mass="${chassis_outer_corner * chassis_outer_thickness * metal_thickness * 4 * metal_density}"
+            x="${chassis_outer_corner}" y="${chassis_outer_thickness}"
+            z="${chassis_outer_thickness}">
+            <origin xyz="0 0 0" rpy="0 0 0" />
+        </xacro:inertial_box>
+    </link>
+    <gazebo reference="frame_right_corner_bottom">
+        <material>Gazebo/White</material>
+    </gazebo>
+    <!-- back corner -->
+    <joint name="frame_back_corner_top_joint" type="fixed">
+        <parent link="center_link" />
+        <child link="frame_back_corner_top" />
+        <origin
+            xyz="-${chassis_length/2 - chassis_empty_space_length/2 + chassis_outer_thickness*135/360} -${chassis_width/2 - chassis_empty_space_width/2 + chassis_outer_thickness*135/360} ${chassis_height + chassis_clearance - chassis_outer_thickness/2}"
+            rpy="0 0 -0.785" />
+    </joint>
+    <link name="frame_back_corner_top">
+        <visual>
+            <geometry>
+                <box size="${chassis_outer_corner} ${chassis_outer_thickness} ${chassis_outer_thickness}" />
+            </geometry>
+            <material name="white" />
+        </visual>
+        <collision>
+            <geometry>
+                <box size="${chassis_outer_corner} ${chassis_outer_thickness} ${chassis_outer_thickness}" />
+            </geometry>
+        </collision>
+        <xacro:inertial_box
+            mass="${chassis_outer_corner * chassis_outer_thickness * metal_thickness * 4 * metal_density}"
+            x="${chassis_outer_corner}" y="${chassis_outer_thickness}"
+            z="${chassis_outer_thickness}">
+            <origin xyz="0 0 0" rpy="0 0 0" />
+        </xacro:inertial_box>
+    </link>
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