Commit message: Robot Base & Level Template

File: src/main_package/description/robot.urdf.xacro (robot description, xacro)
@@ -1,6 +1,9 @@
 <?xml version="1.0"?>
 <robot xmlns:xacro="http://www.ros.org/wiki/xacro" name="robot">
+    <xacro:include filename="inertial_macros.xacro" />
+    <xacro:include filename="materials.xacro" />
     <xacro:include filename="robot_core.xacro" />
     <xacro:include filename="robot_level_1.xacro" />
     <xacro:include filename="robot_level_2.xacro" />
+    <xacro:include filename="robot_level_3.xacro" />
 </robot>

File: src/main_package/description/robot_core.xacro (robot description, xacro)
@@ -1,7 +1,4 @@
 <?xml version="1.0"?>
 <robot xmlns:xacro="http://www.ros.org/wiki/xacro">
-    <!-- INCLUDE -->
-    <xacro:include filename="inertial_macros.xacro" />
-    <xacro:include filename="materials.xacro" />
     <!-- ROBOT PROPERTIES -->
     <xacro:property name="metal_thickness" value="0.003" />
@@ -28,16 +25,9 @@
     <!-- BASE LINK -->
     <link name="base_link"></link>
-    <!-- CENTER LINK -->
-    <joint name="center_joint" type="fixed">
-        <parent link="base_link" />
-        <child link="center_link" />
-        <origin xyz="${chassis_inner_length/2} 0 0" />
-    </joint>
-    <link name="center_link"></link>
     <!-- CHASSIS LINK -->
     <joint name="chassis_joint" type="fixed">
         <parent link="base_link" />
         <child link="chassis" />
-        <origin xyz="${chassis_inner_length/2} 0 0" />
+        <origin xyz="0 0 0" />
     </joint>
     <link name="chassis">
@@ -66,5 +56,5 @@
     <!-- left wheel -->
     <joint name="left_wheel_joint" type="continuous">
-        <parent link="chassis" />
+        <parent link="base_link" />
         <child link="left_wheel" />
         <origin
@@ -94,5 +84,5 @@
     <!-- front wheel -->
     <joint name="front_wheel_joint" type="continuous">
-        <parent link="chassis" />
+        <parent link="base_link" />
         <child link="front_wheel" />
         <origin
@@ -122,5 +112,5 @@
     <!-- right wheel -->
     <joint name="right_wheel_joint" type="continuous">
-        <parent link="chassis" />
+        <parent link="base_link" />
         <child link="right_wheel" />
         <origin
@@ -150,5 +140,5 @@
     <!-- back wheel -->
     <joint name="back_wheel_joint" type="continuous">
-        <parent link="chassis" />
+        <parent link="base_link" />
         <child link="back_wheel" />
         <origin
@@ -182,5 +172,5 @@
     <!-- left corner -->
     <joint name="frame_left_corner_top_joint" type="fixed">
-        <parent link="center_link" />
+        <parent link="base_link" />
         <child link="frame_left_corner_top" />
         <origin
@@ -211,5 +201,5 @@
     </gazebo>
     <joint name="frame_left_corner_bottom_joint" type="fixed">
-        <parent link="center_link" />
+        <parent link="base_link" />
         <child link="frame_left_corner_bottom" />
         <origin
@@ -241,5 +231,5 @@
     <!-- front corner -->
     <joint name="frame_front_corner_top_joint" type="fixed">
-        <parent link="center_link" />
+        <parent link="base_link" />
         <child link="frame_front_corner_top" />
         <origin
@@ -270,5 +260,5 @@
     </gazebo>
     <joint name="frame_front_corner_bottom_joint" type="fixed">
-        <parent link="center_link" />
+        <parent link="base_link" />
         <child link="frame_front_corner_bottom" />
         <origin
@@ -300,5 +290,5 @@
     <!-- right corner -->
     <joint name="frame_right_corner_top_joint" type="fixed">
-        <parent link="center_link" />
+        <parent link="base_link" />
         <child link="frame_right_corner_top" />
         <origin
@@ -329,5 +319,5 @@
     </gazebo>
     <joint name="frame_right_corner_bottom_joint" type="fixed">
-        <parent link="center_link" />
+        <parent link="base_link" />
         <child link="frame_right_corner_bottom" />
         <origin
@@ -359,5 +349,5 @@
     <!-- back corner -->
     <joint name="frame_back_corner_top_joint" type="fixed">
-        <parent link="center_link" />
+        <parent link="base_link" />
         <child link="frame_back_corner_top" />
         <origin
@@ -388,5 +378,5 @@
     </gazebo>
     <joint name="frame_back_corner_bottom_joint" type="fixed">
-        <parent link="center_link" />
+        <parent link="base_link" />
         <child link="frame_back_corner_bottom" />
         <origin
@@ -419,5 +409,5 @@
     <!-- left-front side -->
     <joint name="frame_left_front_side_top_joint" type="fixed">
-        <parent link="center_link" />
+        <parent link="base_link" />
         <child link="frame_left_front_side_top" />
         <origin
@@ -448,5 +438,5 @@
     </gazebo>
     <joint name="frame_left_front_side_bottom_joint" type="fixed">
-        <parent link="center_link" />
+        <parent link="base_link" />
         <child link="frame_left_front_side_bottom" />
         <origin
@@ -478,5 +468,5 @@
     <!-- front-right side -->
     <joint name="frame_front_right_side_top_joint" type="fixed">
-        <parent link="center_link" />
+        <parent link="base_link" />
         <child link="frame_front_right_side_top" />
         <origin
@@ -507,5 +497,5 @@
     </gazebo>
     <joint name="frame_front_right_side_bottom_joint" type="fixed">
-        <parent link="center_link" />
+        <parent link="base_link" />
         <child link="frame_front_right_side_bottom" />
         <origin
@@ -537,5 +527,5 @@
     <!-- right-back side -->
     <joint name="frame_right_back_side_top_joint" type="fixed">
-        <parent link="center_link" />
+        <parent link="base_link" />
         <child link="frame_right_back_side_top" />
         <origin
@@ -566,5 +556,5 @@
     </gazebo>
     <joint name="frame_right_back_side_bottom_joint" type="fixed">
-        <parent link="center_link" />
+        <parent link="base_link" />
         <child link="frame_right_back_side_bottom" />
         <origin
@@ -596,5 +586,5 @@
     <!-- back-left side -->
     <joint name="frame_back_left_side_top_joint" type="fixed">
-        <parent link="center_link" />
+        <parent link="base_link" />
         <child link="frame_back_left_side_top" />
         <origin
@@ -625,5 +615,5 @@
     </gazebo>
     <joint name="frame_back_left_side_bottom_joint" type="fixed">
-        <parent link="center_link" />
+        <parent link="base_link" />
         <child link="frame_back_left_side_bottom" />
         <origin

File: src/main_package/description/robot_level_1.xacro (robot description, xacro)
@@ -1,9 +1,8 @@
 <?xml version="1.0"?>
 <robot xmlns:xacro="http://www.ros.org/wiki/xacro">
-    <!-- INCLUDE -->
-    <xacro:include filename="robot_core.xacro" />
-    <xacro:include filename="inertial_macros.xacro" />
-    <xacro:include filename="materials.xacro" />
     <!-- ROBOT PROPERTIES -->
+    <xacro:property name="support_height" value="0.225" />
+    <xacro:property name="support_radius" value="0.005" />
+    <!-- BASE PLATE -->
     <!-- ARM -->
     <!-- LIDAR -->

File: src/main_package/description/robot_level_2.xacro (robot description, xacro)
@@ -1,8 +1,4 @@
 <?xml version="1.0"?>
 <robot xmlns:xacro="http://www.ros.org/wiki/xacro">
-    <!-- INCLUDE -->
-    <xacro:include filename="robot_core.xacro" />
-    <xacro:include filename="inertial_macros.xacro" />
-    <xacro:include filename="materials.xacro" />
     <!-- ROBOT PROPERTIES -->
     <!-- CPU -->

File: src/main_package/description/robot_level_3.xacro (robot description, xacro)
@@ -1,8 +1,4 @@
 <?xml version="1.0"?>
 <robot xmlns:xacro="http://www.ros.org/wiki/xacro">
-    <!-- INCLUDE -->
-    <xacro:include filename="robot_core.xacro" />
-    <xacro:include filename="inertial_macros.xacro" />
-    <xacro:include filename="materials.xacro" />
     <!-- ROBOT PROPERTIES -->
     <!-- CAMERA -->
