Commit message: Level 1 2 partially done

File: src/main_package/description/robot/robot.urdf.xacro (robot description, xacro)
@@ -2,11 +2,19 @@
 <robot xmlns:xacro="http://www.ros.org/wiki/xacro" name="robot">
     <xacro:property name="package_name" value="main_package" />
+    <!-- SHARED -->
     <xacro:include filename="$(find ${package_name})/description/shared/inertial_macros.xacro" />
     <xacro:include filename="$(find ${package_name})/description/shared/materials.xacro" />
     <xacro:include filename="$(find ${package_name})/description/shared/properties.xacro" />
     <xacro:include filename="$(find ${package_name})/description/shared/supports.urdf.xacro" />
-    <xacro:include filename="$(find ${package_name})/description/robot_core.xacro" />
-    <xacro:include filename="$(find ${package_name})/description/robot_level_1.xacro" />
-    <xacro:include filename="$(find ${package_name})/description/robot_level_2.xacro" />
-    <xacro:include filename="$(find ${package_name})/description/robot_level_3.xacro" />
+    <!-- FUNCTIONAL -->
+    <xacro:include filename="$(find ${package_name})/description/functional/depth_camera.urdf.xacro" />
+    <xacro:include filename="$(find ${package_name})/description/functional/display.urdf.xacro" />
+    <xacro:include filename="$(find ${package_name})/description/functional/lidar.urdf.xacro" />
+    <xacro:include filename="$(find ${package_name})/description/functional/mic.urdf.xacro" />
+    <xacro:include filename="$(find ${package_name})/description/functional/stop_button.urdf.xacro" />
+    <!-- ROBOT -->
+    <xacro:include filename="$(find ${package_name})/description/robot/robot_core.xacro" />
+    <xacro:include filename="$(find ${package_name})/description/robot/robot_level_1.xacro" />
+    <xacro:include filename="$(find ${package_name})/description/robot/robot_level_2.xacro" />
+    <xacro:include filename="$(find ${package_name})/description/robot/robot_level_3.xacro" />
 </robot>

File: src/main_package/description/robot/robot_core.xacro (robot description, xacro)
@@ -78,5 +78,5 @@
                 <cylinder radius="${wheel_radius}" length="${wheel_thickness}" />
             </geometry>
-            <material name="red" />
+            <material name="blue" />
         </visual>
         <collision>
@@ -90,5 +90,5 @@
     </link>
     <gazebo reference="front_wheel">
-        <material>Gazebo/Red</material>
+        <material>Gazebo/Blue</material>
     </gazebo>
     <!-- right wheel -->
@@ -151,5 +151,6 @@
     <!-- CORNERS -->
     <!-- left corner -->
-    <xacro:corner_frame nameprefix="frame_left_corner_top" bx="${chassis_outer_corner}" by="${chassis_outer_thickness}"
+    <xacro:corner_frame nameprefix="frame_left_corner_top" parent="base_link" bx="${chassis_outer_corner}"
+        by="${chassis_outer_thickness}"
         bz="${chassis_outer_thickness}">
         <origin
@@ -157,5 +158,5 @@
             rpy="0 0 0.785" />
     </xacro:corner_frame>
-    <xacro:corner_frame nameprefix="frame_left_corner_bottom" bx="${chassis_outer_corner}"
+    <xacro:corner_frame nameprefix="frame_left_corner_bottom" parent="base_link" bx="${chassis_outer_corner}"
         by="${chassis_outer_thickness}" bz="${chassis_outer_thickness}">
         <origin
@@ -164,5 +165,6 @@
     </xacro:corner_frame>
     <!-- front corner -->
-    <xacro:corner_frame nameprefix="frame_front_corner_top" bx="${chassis_outer_corner}" by="${chassis_outer_thickness}"
+    <xacro:corner_frame nameprefix="frame_front_corner_top" parent="base_link" bx="${chassis_outer_corner}"
+        by="${chassis_outer_thickness}"
         bz="${chassis_outer_thickness}">
         <origin
@@ -170,5 +172,5 @@
             rpy="0 0 -0.785" />
     </xacro:corner_frame>
-    <xacro:corner_frame nameprefix="frame_front_corner_bottom" bx="${chassis_outer_corner}"
+    <xacro:corner_frame nameprefix="frame_front_corner_bottom" parent="base_link" bx="${chassis_outer_corner}"
         by="${chassis_outer_thickness}" bz="${chassis_outer_thickness}">
         <origin
@@ -177,5 +179,6 @@
     </xacro:corner_frame>
     <!-- right corner -->
-    <xacro:corner_frame nameprefix="frame_right_corner_top" bx="${chassis_outer_corner}" by="${chassis_outer_thickness}"
+    <xacro:corner_frame nameprefix="frame_right_corner_top" parent="base_link" bx="${chassis_outer_corner}"
+        by="${chassis_outer_thickness}"
         bz="${chassis_outer_thickness}">
         <origin
@@ -183,5 +186,5 @@
             rpy="0 0 0.785" />
     </xacro:corner_frame>
-    <xacro:corner_frame nameprefix="frame_right_corner_bottom" bx="${chassis_outer_corner}"
+    <xacro:corner_frame nameprefix="frame_right_corner_bottom" parent="base_link" bx="${chassis_outer_corner}"
         by="${chassis_outer_thickness}" bz="${chassis_outer_thickness}">
         <origin
@@ -190,5 +193,6 @@
     </xacro:corner_frame>
     <!-- back corner -->
-    <xacro:corner_frame nameprefix="frame_back_corner_top" bx="${chassis_outer_corner}" by="${chassis_outer_thickness}"
+    <xacro:corner_frame nameprefix="frame_back_corner_top" parent="base_link" bx="${chassis_outer_corner}"
+        by="${chassis_outer_thickness}"
         bz="${chassis_outer_thickness}">
         <origin
@@ -196,5 +200,5 @@
             rpy="0 0 -0.785" />
     </xacro:corner_frame>
-    <xacro:corner_frame nameprefix="frame_back_corner_bottom" bx="${chassis_outer_corner}"
+    <xacro:corner_frame nameprefix="frame_back_corner_bottom" parent="base_link" bx="${chassis_outer_corner}"
         by="${chassis_outer_thickness}" bz="${chassis_outer_thickness}">
         <origin

File: src/main_package/description/shared/materials.xacro (robot description, xacro)
@@ -1,30 +1,43 @@
 <?xml version="1.0"?>
 <robot xmlns:xacro="http://www.ros.org/wiki/xacro">
+    <!-- DISPLAY -->
     <material name="black">
         <color rgba="0 0 0 1" />
     </material>
+    <!-- SUPPORT -->
+    <material name="grey">
+        <color rgba="0.5 0.5 0.5 1" />
+    </material>
+    <!-- MIC -->
+    <material name="dark_grey">
+        <color rgba="0.25 0.25 0.25 1" />
+    </material>
+    <!-- MIC -->
+    <material name="orange">
+        <color rgba="1 0.3 0.1 1" />
+    </material>
+    <!-- FRAME -->
     <material name="white">
         <color rgba="1 1 1 1" />
     </material>
+    <!-- BASE PLATE -->
     <material name="white_transparent">
         <color rgba="1 1 1 0.5" />
     </material>
+    <!-- STOP BUTTON -->
     <material name="red">
         <color rgba="1 0 0 1" />
     </material>
+    <!-- CPU -->
     <material name="green">
         <color rgba="0.2 1 0.2 1" />
     </material>
+    <!-- WHEEL -->
     <material name="blue">
         <color rgba="0.2 0.2 1 1" />
     </material>
+    <!-- CAMERA -->
     <material name="yellow">
         <color rgba="1 1 0.6 1" />
     </material>
-    <material name="teal">
-        <color rgba="0.2 0.8 0.7 1" />
-    </material>
-    <material name="raspberry">
-        <color rgba="0.7 0.1 0.4 1" />
-    </material>
 </robot>

File: src/main_package/description/shared/properties.xacro (robot description, xacro)
@@ -1,4 +1,9 @@
 <?xml version="1.0"?>
 <robot xmlns:xacro="http://www.ros.org/wiki/xacro">
+    <!--
+        LENGTH: x
+        WIDTH: y
+        HEIGHT: z
+    -->
     <!-- ROBOT CORE PROPERTIES -->
     <xacro:property name="metal_thickness" value="0.003" />
@@ -15,4 +20,5 @@
     <xacro:property name="chassis_outer_side" value="0.272" />
     <xacro:property name="chassis_outer_corner" value="0.162" />
+    <xacro:property name="chassis_corner_margin" value="0.080" />
     <xacro:property name="chassis_outer_thickness" value="0.020" />
     <xacro:property name="chassis_height" value="0.120" />
@@ -22,4 +28,6 @@
     <!-- ROBOT LEVEL 1 PROPERTIES -->
     <xacro:property name="level_1_height_displacement" value="${chassis_clearance + chassis_height}" />
+    <xacro:property name="level_1_length_displacement" value="0.000" />
+    <xacro:property name="level_1_width_displacement" value="0.000" />
     <xacro:property name="level_1_base_length" value="0.500" />
     <xacro:property name="level_1_base_width" value="0.500" />
@@ -32,27 +40,96 @@
     <xacro:property name="level_1_empty_space_length" value="${(level_1_base_length - chassis_outer_thickness*4)/3}" />
     <xacro:property name="level_1_empty_space_width" value="${(level_1_base_width - chassis_outer_thickness*4)/3}" />
+    <xacro:property name="level_1_center_x"
+        value="${-chassis_length/2 + level_1_length_displacement + level_1_base_length/2}" />
+    <xacro:property name="level_1_center_y"
+        value="${-chassis_width/2 + level_1_width_displacement + level_1_base_width/2}" />
+    <xacro:property name="level_1_center_z"
+        value="${level_1_height_displacement + metal_thickness}" />
     <!-- ROBOT LEVEL 2 PROPERTIES -->
     <xacro:property name="level_2_height_displacement"
         value="${level_1_height_displacement + metal_thickness + level_1_support_height}" />
-    <xacro:property name="level_2_length_displacement" value="0.010" />
+    <xacro:property name="level_2_length_displacement" value="0.020" />
+    <xacro:property name="level_2_width_displacement" value="0.020" />
     <xacro:property name="level_2_base_length" value="0.475" />
     <xacro:property name="level_2_base_width" value="0.475" />
     <xacro:property name="level_2_support_height" value="0.253" />
     <xacro:property name="level_2_support_radius" value="0.0075" />
-    <xacro:property name="level_2_support_displacement_x" value="${level_2_base_length/8}" />
-    <xacro:property name="level_2_support_displacement_y" value="${level_2_base_width/8}" />
+    <xacro:property name="level_2_support_displacement_x"
+        value="${(level_2_base_length + chassis_corner_margin)/8}" />
+    <xacro:property name="level_2_support_displacement_y"
+        value="${(level_2_base_width + chassis_corner_margin)/8}" />
     <xacro:property name="level_2_corner_length" value="${chassis_outer_corner * level_2_base_length / chassis_length}" />
     <xacro:property name="level_2_corner_width" value="${chassis_outer_corner * level_2_base_width / chassis_width}" />
     <xacro:property name="level_2_empty_space_length" value="${(level_2_base_length - chassis_outer_thickness*4)/3}" />
     <xacro:property name="level_2_empty_space_width" value="${(level_2_base_width - chassis_outer_thickness*4)/3}" />
+    <xacro:property name="level_2_center_x"
+        value="${-chassis_length/2 + level_2_length_displacement + level_2_base_length/2}" />
+    <xacro:property name="level_2_center_y"
+        value="${-chassis_width/2 + level_2_width_displacement + level_2_base_width/2}" />
+    <xacro:property name="level_2_center_z"
+        value="${level_2_height_displacement + metal_thickness}" />
+    <!-- CPU -->
+    <xacro:property name="cpu_length" value="0.105" />
+    <xacro:property name="cpu_width" value="0.145" />
+    <xacro:property name="cpu_height" value="0.040" />
+    <xacro:property name="cpu_weight" value="0.400" />
+    <xacro:property name="cpu_offset_x" value="-0.070" />
+    <xacro:property name="cpu_offset_y" value="-0.090" />
+    <!-- NETWORK INTERFACE -->
+    <xacro:property name="network_length" value="0.150" />
+    <xacro:property name="network_width" value="0.060" />
+    <xacro:property name="network_height" value="0.030" />
+    <xacro:property name="network_weight" value="0.150" />
+    <xacro:property name="network_offset_x" value="-0.070" />
+    <xacro:property name="network_offset_y" value="0.040" />
     <!-- ROBOT LEVEL 3 PROPERTIES -->
     <xacro:property name="level_3_height_displacement"
         value="${level_2_height_displacement + metal_thickness + level_2_support_height}" />
-    <xacro:property name="level_3_length_displacement" value="0.040" />
+    <xacro:property name="level_3_length_displacement" value="0.065" />
+    <xacro:property name="level_3_width_displacement" value="0.114" />
     <xacro:property name="level_3_base_length" value="0.240" />
     <xacro:property name="level_3_base_width" value="0.272" />
-    <xacro:property name="level_3_support_height" value="0.253" />
+    <xacro:property name="level_3_support_height" value="0.252" />
     <xacro:property name="level_3_support_radius" value="0.0075" />
     <xacro:property name="level_3_support_displacement_x" value="${level_3_base_length/8}" />
     <xacro:property name="level_3_support_displacement_y" value="${level_3_base_width/8}" />
+    <xacro:property name="level_3_center_x"
+        value="${-chassis_length/2 + level_3_length_displacement + level_3_base_length/2}" />
+    <xacro:property name="level_3_center_y"
+        value="${-chassis_width/2 + level_3_width_displacement + level_3_base_width/2}" />
+    <xacro:property name="level_3_center_z"
+        value="${level_3_height_displacement + metal_thickness}" />
+    <!-- DEPTH CAMERA -->
+    <!-- NAME | x y z | weight | fixture_radius fixture_length -->
+    <!-- intel REALSENSE | 0.026 0.124 0.029 | 0.38 | 0.0125 0.073 -->
+    <xacro:property name="intel_camera_length" value="0.026" />
+    <xacro:property name="intel_camera_width" value="0.124" />
+    <xacro:property name="intel_camera_height" value="0.029" />
+    <xacro:property name="intel_camera_and_fixture_weight" value="0.380" />
+    <xacro:property name="intel_camera_fixture_radius" value="0.0125" />
+    <xacro:property name="intel_camera_fixture_length" value="0.073" />
+    <!-- DISPLAY -->
+    <xacro:property name="display_length" value="0.015" />
+    <xacro:property name="display_width" value="0.235" />
+    <xacro:property name="display_height" value="0.145" />
+    <xacro:property name="display_weight" value="0.97" />
+    <xacro:property name="display_support_radius" value="0.0075" />
+    <xacro:property name="display_support_height" value="0.252" />
+    <xacro:property name="display_offset_x" value="-0.100" />
+    <xacro:property name="display_offset_y" value="0.055" />
+    <!-- MIC -->
+    <xacro:property name="mic_base_length" value="0.010" />
+    <xacro:property name="mic_base_radius" value="0.036" />
+    <xacro:property name="mic_support_length" value="0.070" />
+    <xacro:property name="mic_support_radius" value="0.005" />
+    <xacro:property name="mic_length" value="0.150" />
+    <xacro:property name="mic_radius" value="0.015" />
+    <xacro:property name="mic_weight" value="0.200" />
+    <xacro:property name="mic_offset_x" value="0.030" />
+    <xacro:property name="mic_offset_y" value="0.070" />
+    <!-- STOP BUTTON -->
+    <xacro:property name="stop_button_radius" value="0.018" />
+    <xacro:property name="stop_button_length" value="0.030" />
+    <xacro:property name="stop_button_weight" value="0.046" />
+    <xacro:property name="stop_button_offset_y" value="0.080" />
 </robot>

File: src/main_package/description/shared/supports.urdf.xacro (robot description, xacro)
@@ -2,11 +2,11 @@
 <robot xmlns:xacro="http://www.ros.org/wiki/xacro">
     <!-- BASE CORNER -->
-    <xacro:macro name="corner_frame" params="nameprefix bx by bz *origin">
+    <xacro:macro name="corner_frame" params="nameprefix parent bx by bz *origin">
         <joint name="${nameprefix}_joint" type="fixed">
-            <parent link="base_link" />
-            <child link="${nameprefix}" />
+            <parent link="${parent}" />
+            <child link="${nameprefix}_link" />
             <xacro:insert_block name="origin" />
         </joint>
-        <link name="${nameprefix}">
+        <link name="${nameprefix}_link">
             <visual>
                 <geometry>
@@ -27,5 +27,5 @@
             </xacro:inertial_box>
         </link>
-        <gazebo reference="${nameprefix}">
+        <gazebo reference="${nameprefix}_link">
             <material>Gazebo/White</material>
         </gazebo>
@@ -35,8 +35,8 @@
         <joint name="${nameprefix}_joint" type="fixed">
             <parent link="base_link" />
-            <child link="${nameprefix}" />
+            <child link="${nameprefix}_link" />
             <xacro:insert_block name="origin" />
         </joint>
-        <link name="${nameprefix}">
+        <link name="${nameprefix}_link">
             <visual>
                 <geometry>
@@ -57,21 +57,21 @@
             </xacro:inertial_box>
         </link>
-        <gazebo reference="${nameprefix}">
+        <gazebo reference="${nameprefix}_link">
             <material>Gazebo/White</material>
         </gazebo>
     </xacro:macro>
     <!-- SUPPORT CYLINDER -->
-    <xacro:macro name="support_cylinder" params="nameprefix length radius *origin">
+    <xacro:macro name="support_cylinder" params="nameprefix parent length radius *origin">
         <joint name="${nameprefix}_joint" type="fixed">
-            <parent link="base_link" />
-            <child link="${nameprefix}" />
+            <parent link="${parent}" />
+            <child link="${nameprefix}_link" />
             <xacro:insert_block name="origin" />
         </joint>
-        <link name="${nameprefix}">
+        <link name="${nameprefix}_link">
             <visual>
                 <geometry>
                     <cylinder radius="${radius}" length="${length}" />
                 </geometry>
-                <material name="white" />
+                <material name="grey" />
             </visual>
             <collision>
@@ -86,16 +86,16 @@
             </xacro:inertial_cylinder>
         </link>
-        <gazebo reference="${nameprefix}">
+        <gazebo reference="${nameprefix}_link">
             <material>Gazebo/Grey</material>
         </gazebo>
     </xacro:macro>
     <!-- BASE PLATE -->
-    <xacro:macro name="base_plate" params="nameprefix bx by bz *origin">
+    <xacro:macro name="base_plate" params="nameprefix parent bx by bz *origin">
         <joint name="${nameprefix}_joint" type="fixed">
-            <parent link="base_link" />
-            <child link="${nameprefix}" />
+            <parent link="${parent}" />
+            <child link="${nameprefix}_link" />
             <xacro:insert_block name="origin" />
         </joint>
-        <link name="${nameprefix}">
+        <link name="${nameprefix}_link">
             <visual>
                 <geometry>
@@ -116,5 +116,5 @@
             </xacro:inertial_box>
         </link>
-        <gazebo reference="${nameprefix}">
+        <gazebo reference="${nameprefix}_link">
             <material>Gazebo/White</material>
         </gazebo>
