Commit message: integrated rviz gazebo into simulation launch

File: src/main_package/description/functional/depth_camera.urdf.xacro (robot description, xacro)
@@ -2,5 +2,5 @@
 <robot xmlns:xacro="http://www.ros.org/wiki/xacro">
     <xacro:macro name="depth_camera"
-        params="nameprefix parent camera_length camera_width camera_height mass fixture_radius fixture_length *origin">
+        params="nameprefix parent camera_length camera_width camera_height mass fixture_radius fixture_length *origin *frame_name">
         <!-- CAMERA FIXTURE -->
         <joint name="${nameprefix}_fixture_joint" type="fixed">
@@ -48,5 +48,5 @@
             <parent link="${nameprefix}_link" />
             <child link="${nameprefix}_link_optical" />
-            <origin xyz="0 0 0" rpy="${pi/2} 0 ${-pi/2}" />
+            <origin xyz="0 0 0" rpy="${-pi/2} 0 ${-pi/2}" />
         </joint>
         <link name="${nameprefix}_link_optical"></link>
@@ -71,5 +71,6 @@
                 </camera>
                 <plugin name="${nameprefix}_controller" filename="libgazebo_ros_camera.so">
-                    <frame_name>camera_link_optical</frame_name>
+                    <!-- <frame_name>camera_link_optical</frame_name> -->
+                    <xacro:insert_block name="frame_name" />
                     <min_depth>0.1</min_depth>
                     <max_depth>100.0</max_depth>

File: src/main_package/description/functional/lidar.urdf.xacro (robot description, xacro)
@@ -1,2 +1,59 @@
 <?xml version="1.0"?>
-<robot xmlns:xacro="http://www.ros.org/wiki/xacro"></robot>
+<robot xmlns:xacro="http://www.ros.org/wiki/xacro">
+    <xacro:macro name="lidar" params="nameprefix parent length radius mass *origin *frame_name">
+        <joint name="${nameprefix}_joint" type="fixed">
+            <parent link="${parent}" />
+            <child link="${nameprefix}_frame" />
+            <xacro:insert_block name="origin" />
+        </joint>
+        <link name="${nameprefix}_frame">
+            <visual>
+                <geometry>
+                    <cylinder length="${length}" radius="${radius}" />
+                </geometry>
+                <material name="purple" />
+            </visual>
+            <collision>
+                <geometry>
+                    <cylinder length="${length}" radius="${radius}" />
+                </geometry>
+            </collision>
+            <xacro:inertial_cylinder
+                mass="${mass}"
+                length="${length}" radius="${radius}">
+                <origin xyz="0 0 0" rpy="0 0 0" />
+            </xacro:inertial_cylinder>
+        </link>
+        <gazebo reference="${nameprefix}_frame">
+            <material>Gazebo/Purple</material>
+            <sensor name="${nameprefix}" type="ray">
+                <pose> 0 0 0 0 0 0 </pose>
+                <visualize>true</visualize>
+                <update_rate>10</update_rate>
+                <ray>
+                    <scan>
+                        <horizontal>
+                            <sample>360</sample>
+                            <resolution>1</resolution>
+                            <min_angle>-3.14</min_angle>
+                            <max_angle>3.14</max_angle>
+                        </horizontal>
+                    </scan>
+                    <range>
+                        <min>0.3</min>
+                        <max>12</max>
+                        <resolution>0.01</resolution>
+                    </range>
+                </ray>
+                <plugin name="${nameprefix}_controller" filename="libgazebo_ros_ray_sensor.so">
+                    <ros>
+                        <argument>~/out:=scan</argument>
+                    </ros>
+                    <output_type>sensor_msgs/LaserScan</output_type>
+                    <!-- <frame_name>laser_frame</frame_name> -->
+                    <xacro:insert_block name="frame_name" />
+                </plugin>
+            </sensor>
+        </gazebo>
+    </xacro:macro>
+</robot>

File: src/main_package/description/robot/robot_level_1.xacro (robot description, xacro)
@@ -22,6 +22,13 @@
     <link name="level_1_center_link">
     </link>
-    <!-- ARM -->
     <!-- LIDAR -->
+    <xacro:lidar nameprefix="laser"
+        parent="level_1_center_link"
+        length="${lidar_length}"
+        radius="${lidar_radius}"
+        mass="${lidar_weight}">
+        <origin xyz="0 0 ${lidar_length/2}" rpy="0 0 0" />
+        <frame_name>laser_frame</frame_name>
+    </xacro:lidar>
     <!-- BASE PLATE -->
     <xacro:base_plate nameprefix="level_1_base_plate_x"

File: src/main_package/description/robot/robot_level_2.xacro (robot description, xacro)
@@ -22,4 +22,5 @@
     <link name="level_2_center_link">
     </link>
+    <!-- ARM -->
     <!-- CPU -->
     <joint name="$cpu_joint" type="fixed">

File: src/main_package/description/robot/robot_level_3.xacro (robot description, xacro)
@@ -66,4 +66,5 @@
         fixture_length="${intel_camera_fixture_length}">
         <origin xyz="0 0 ${intel_camera_fixture_length/2}" rpy="0 0 0" />
+        <frame_name>camera_1_link_optical</frame_name>
     </xacro:depth_camera>
     <xacro:depth_camera nameprefix="camera_2"
@@ -77,4 +78,5 @@
         <origin xyz="${level_3_base_length/2 - intel_camera_fixture_radius} 0 ${intel_camera_fixture_length/2}"
             rpy="0 0 0" />
+        <frame_name>camera_2_link_optical</frame_name>
     </xacro:depth_camera>
     <!-- MIC -->

File: src/main_package/description/shared/materials.xacro (robot description, xacro)
@@ -41,3 +41,7 @@
         <color rgba="1 1 0.6 1" />
     </material>
+    <!-- LIDAR -->
+    <material name="purple">
+        <color rgba="0.627 0.125 0.941 1" />
+    </material>
 </robot>

File: src/main_package/description/shared/properties.xacro (robot description, xacro)
@@ -46,4 +46,8 @@
     <xacro:property name="level_1_center_z"
         value="${level_1_height_displacement + metal_thickness}" />
+    <!-- LIDAR -->
+    <xacro:property name="lidar_radius" value="0.030" />
+    <xacro:property name="lidar_length" value="0.068" />
+    <xacro:property name="lidar_weight" value="0.400" />
     <!-- ROBOT LEVEL 2 PROPERTIES -->
     <xacro:property name="level_2_height_displacement"

Commit message: wheel calibration done

File: src/main_package/description/functional/depth_camera.urdf.xacro (robot description, xacro)
@@ -52,5 +52,5 @@
         <link name="${nameprefix}_link_optical"></link>
         <!-- GAZEBO CONFIG -->
-        <gazebo reference="${nameprefix}_link">
+        <!-- <gazebo reference="${nameprefix}_link">
             <material>Gazebo/Yellow</material>
             <sensor name="${nameprefix}" type="depth">
@@ -76,4 +76,34 @@
                 </plugin>
             </sensor>
+        </gazebo> -->
+        <gazebo reference="${nameprefix}_link">
+            <sensor name="${nameprefix}_link" type="camera">
+                <update_rate>10.0</update_rate>
+                <always_on>true</always_on>
+                <ignition_frame_id>${nameprefix}_link</ignition_frame_id>
+                <pose>0 0 0 0 0 0</pose>
+                <topic>/${nameprefix}/image_raw</topic>
+                <camera name="${nameprefix}">
+                    <!--
+                <triggered>true</triggered>
+                <trigger_topic>/trigger</trigger_topic>
+                -->
+                    <horizontal_fov>1.0</horizontal_fov>
+                    <image>
+                        <width>1280</width>
+                        <height>720</height>
+                        <format>R8G8B8</format>
+                    </image>
+                    <clip>
+                        <near>0.02</near>
+                        <far>8</far>
+                    </clip>
+                </camera>
+                <!-- <plugin name="${nameprefix}_controller" filename="libgazebo_ros_camera.so">
+                    <frame_name>${nameprefix}_link_optical</frame_name>
+                    <min_depth>0.1</min_depth>
+                    <max_depth>100.0</max_depth>
+                </plugin> -->
+            </sensor>
         </gazebo>
     </xacro:macro>

File: src/main_package/description/functional/lidar.urdf.xacro (robot description, xacro)
@@ -48,5 +48,6 @@
                 <plugin name="${nameprefix}_controller" filename="libgazebo_ros_ray_sensor.so">
                     <ros>
-                        <argument>--ros-args --remap ~/out:=scan</argument>
+                        <!-- <argument>ros-args remap ~/out:=scan</argument> -->
+                        <argument>~/out:=scan</argument>
                     </ros>
                     <output_type>sensor_msgs/LaserScan</output_type>

File: src/main_package/description/gazebo/robot_gazebo.gazebo.xacro (robot description, xacro)
@@ -4,7 +4,5 @@
     <!-- =============== Gazebo =============== -->
     <gazebo>
-      <!--
-      <plugin filename="gz_ros2_control-system" name="gz_ros2_control::GazeboSimROS2ControlPlugin">
-      -->
+      <!-- <plugin filename="gz_ros2_control-system" name="gz_ros2_control::GazeboSimROS2ControlPlugin"> -->
       <plugin filename="ign_ros2_control-system" name="ign_ros2_control::IgnitionROS2ControlPlugin">
         <parameters>$(find main_package)/config/robot_config.yaml</parameters>

File: src/main_package/description/robot/robot_core.xacro (robot description, xacro)
@@ -38,4 +38,5 @@
             xyz="-${chassis_inner_length/2 + wheel_thickness/2} ${chassis_inner_width/2 + wheel_thickness/2} ${wheel_radius/2}"
             rpy="0 ${pi/2} ${pi*3/4}" />
+        <!-- <origin xyz="-0.35 0.35 0.05" rpy="0 ${pi/2} ${pi*3/4}" /> -->
     </xacro:omni_wheel>
     <!-- <joint name="left_wheel_joint" type="continuous">
@@ -73,4 +74,5 @@
             xyz="${chassis_inner_length/2 + wheel_thickness/2} ${chassis_inner_width/2 + wheel_thickness/2} ${wheel_radius/2}"
             rpy="0 ${pi/2} ${pi/4}" />
+        <!-- <origin xyz="0.35 0.35 0.05" rpy="0 ${pi/2} ${pi/4}" /> -->
     </xacro:omni_wheel>
     <!-- <joint name="front_wheel_joint" type="continuous">
@@ -103,8 +105,9 @@
     <!-- right wheel -->
     <!-- Wheel3 -->
-    <xacro:omni_wheel prefix="wheel2" parent="base_link">
-        <origin
-            xyz="${chassis_inner_length/2 + wheel_thickness/2} -${chassis_inner_width/2 + wheel_thickness/2} ${wheel_radius/2}"
+    <xacro:omni_wheel prefix="wheel3" parent="base_link">
+        <origin
+            xyz="-${chassis_inner_length/2 + wheel_thickness/2} -${chassis_inner_width/2 + wheel_thickness/2} ${wheel_radius/2}"
             rpy="0 ${pi/2} ${-pi*3/4}" />
+        <!-- <origin xyz="-0.35 -0.35 0.05" rpy="0 ${pi/2} ${-pi*3/4}" /> -->
     </xacro:omni_wheel>
     <!-- <joint name="right_wheel_joint" type="continuous">
@@ -137,8 +140,9 @@
     <!-- back wheel -->
     <!-- Wheel2 -->
-    <xacro:omni_wheel prefix="wheel3" parent="base_link">
-        <origin
-            xyz="-${chassis_inner_length/2 + wheel_thickness/2} -${chassis_inner_width/2 + wheel_thickness/2} ${wheel_radius/2}"
+    <xacro:omni_wheel prefix="wheel2" parent="base_link">
+        <origin
+            xyz="${chassis_inner_length/2 + wheel_thickness/2} -${chassis_inner_width/2 + wheel_thickness/2} ${wheel_radius/2}"
             rpy="0 ${pi/2} ${-pi/4}" />
+        <!-- <origin xyz="0.35 -0.35 0.05" rpy="0 ${pi/2} ${-pi/4}" /> -->
     </xacro:omni_wheel>
     <!-- <joint name="back_wheel_joint" type="continuous">

File: src/main_package/description/ros2_control/robot_ros2.ros2_control.xacro (robot description, xacro)
@@ -11,7 +11,5 @@
         </xacro:if>
         <xacro:if value="${use_sim}">
-          <!--
-          <plugin>gz_ros2_control/GazeboSimSystem</plugin>
-         -->
+          <!-- <plugin>gz_ros2_control/GazeboSimSystem</plugin> -->
           <plugin>ign_ros2_control/IgnitionSystem</plugin>
         </xacro:if>

File: src/main_package/description/shared/properties.xacro (robot description, xacro)
@@ -16,4 +16,5 @@
     <xacro:property name="wheel_radius" value="0.050" />
     <xacro:property name="wheel_thickness" value="0.038" />
+    <xacro:property name="wheel_padding" value="0.005" />
     <!-- CHASSIS & FRAME PROPS -->
     <xacro:property name="chassis_length" value="0.500" />
@@ -26,5 +27,5 @@
     <xacro:property name="chassis_outer_thickness" value="0.020" />
     <xacro:property name="chassis_height" value="0.120" />
-    <xacro:property name="chassis_clearance" value="0.030" />
+    <xacro:property name="chassis_clearance" value="0.050" />
     <xacro:property name="chassis_empty_space_length" value="${(chassis_length - chassis_outer_thickness*4)/3}" />
     <xacro:property name="chassis_empty_space_width" value="${(chassis_width - chassis_outer_thickness*4)/3}" />
