Commit message: model showing  need to fix speed issues

File: src/main_package/description/functional/depth_camera.urdf.xacro (robot description, xacro)
@@ -3,5 +3,4 @@
     <xacro:macro name="depth_camera"
         params="nameprefix parent camera_length camera_width camera_height mass fixture_radius fixture_length *origin">
-        <!-- CAMERA FIXTURE -->
         <joint name="${nameprefix}_fixture_joint" type="fixed">
             <parent link="${parent}" />
@@ -30,5 +29,4 @@
             <material>Gazebo/Grey</material>
         </gazebo>
-        <!-- GAZEBO CAMERA -->
         <joint name="${nameprefix}_joint" type="fixed">
             <parent link="${nameprefix}_fixture_link" />
@@ -44,5 +42,4 @@
             </visual>
         </link>
-        <!-- ROS2 CAMERA -->
         <joint name="${nameprefix}_optical_joint" type="fixed">
             <parent link="${nameprefix}_link" />
@@ -51,6 +48,5 @@
         </joint>
         <link name="${nameprefix}_link_optical"></link>
-        <!-- GAZEBO CONFIG -->
-        <!-- <gazebo reference="${nameprefix}_link">
+        <gazebo reference="${nameprefix}_link">
             <material>Gazebo/Yellow</material>
             <sensor name="${nameprefix}" type="depth">
@@ -76,34 +72,4 @@
                 </plugin>
             </sensor>
-        </gazebo> -->
-        <gazebo reference="${nameprefix}_link">
-            <sensor name="${nameprefix}_link" type="camera">
-                <update_rate>10.0</update_rate>
-                <always_on>true</always_on>
-                <ignition_frame_id>${nameprefix}_link</ignition_frame_id>
-                <pose>0 0 0 0 0 0</pose>
-                <topic>/${nameprefix}/image_raw</topic>
-                <camera name="${nameprefix}">
-                    <!--
-                <triggered>true</triggered>
-                <trigger_topic>/trigger</trigger_topic>
-                -->
-                    <horizontal_fov>1.0</horizontal_fov>
-                    <image>
-                        <width>1280</width>
-                        <height>720</height>
-                        <format>R8G8B8</format>
-                    </image>
-                    <clip>
-                        <near>0.02</near>
-                        <far>8</far>
-                    </clip>
-                </camera>
-                <!-- <plugin name="${nameprefix}_controller" filename="libgazebo_ros_camera.so">
-                    <frame_name>${nameprefix}_link_optical</frame_name>
-                    <min_depth>0.1</min_depth>
-                    <max_depth>100.0</max_depth>
-                </plugin> -->
-            </sensor>
         </gazebo>
     </xacro:macro>

File: src/main_package/description/functional/lidar.urdf.xacro (robot description, xacro)
@@ -48,9 +48,7 @@
                 <plugin name="${nameprefix}_controller" filename="libgazebo_ros_ray_sensor.so">
                     <ros>
-                        <!-- <argument>ros-args remap ~/out:=scan</argument> -->
                         <argument>~/out:=scan</argument>
                     </ros>
                     <output_type>sensor_msgs/LaserScan</output_type>
-                    <!-- <frame_name>laser_frame</frame_name> -->
                     <xacro:insert_block name="frame_name" />
                 </plugin>

File: src/main_package/description/functional/mic.urdf.xacro (robot description, xacro)
@@ -3,5 +3,4 @@
     <xacro:macro name="mic"
         params="nameprefix parent base_length base_radius support_length support_radius mic_length mic_radius mass *origin">
-        <!-- base -->
         <joint name="${nameprefix}_base_joint" type="fixed">
             <parent link="${parent}" />
@@ -30,5 +29,4 @@
             <material>Gazebo/DarkGrey</material>
         </gazebo>
-        <!-- support -->
         <joint name="${nameprefix}_support_joint" type="fixed">
             <parent link="${nameprefix}_base_link" />
@@ -57,5 +55,4 @@
             <material>Gazebo/DarkGrey</material>
         </gazebo>
-        <!-- MIC -->
         <joint name="${nameprefix}_joint" type="fixed">
             <parent link="${nameprefix}_support_link" />

File: src/main_package/description/functional/wheel/wheel.urdf.xacro (robot description, xacro)
@@ -85,5 +85,4 @@
     <link name="${prefix}_housing_s_link">
       <inertial>
-        <!-- Links without mass cannot be used in gazebo. -->
         <mass value="0.001" />
         <inertia ixx="0" ixy="0" ixz="0" iyy="0" iyz="0" izz="0.00001" />

File: src/main_package/description/functional/wheel/wheel_100mm.urdf.xacro (robot description, xacro)
@@ -85,5 +85,4 @@
     <link name="${prefix}_housing_s_link">
       <inertial>
-        <!-- Links without mass cannot be used in gazebo. -->
         <mass value="0.001" />
         <inertia ixx="0" ixy="0" ixz="0" iyy="0" iyz="0" izz="0.00001" />

File: src/main_package/description/gazebo/robot_gazebo.gazebo.xacro (robot description, xacro)
@@ -2,11 +2,11 @@
 <robot xmlns:xacro="http://ros.org/wiki/xacro">
   <xacro:macro name="robot_gazebo" params="prefix">
-    <!-- =============== Gazebo =============== -->
     <gazebo>
-      <!-- <plugin filename="gz_ros2_control-system" name="gz_ros2_control::GazeboSimROS2ControlPlugin"> -->
-      <plugin filename="ign_ros2_control-system" name="ign_ros2_control::IgnitionROS2ControlPlugin">
+      <plugin name="gazebo_ros2_control" filename="libgazebo_ros2_control.so">
+        <robotNamespace>/</robotNamespace>
         <parameters>$(find main_package)/config/robot_config.yaml</parameters>
+        <parameters>$(find main_package)/params/gaz_ros2_ctl_use_sim.yaml</parameters>
       </plugin>
-      <plugin filename="ignition-gazebo-sensors-system" name="ignition::gazebo::systems::Sensors">
+      <plugin name="gazebo_ros_sensors" filename="libgazebo_ros_sensors.so">
         <render_engine>ogre2</render_engine>
       </plugin>

File: src/main_package/description/robot/robot.urdf.xacro (robot description, xacro)
@@ -4,10 +4,8 @@
     <xacro:arg name="use_sim" default="false" />
     <xacro:property name="package_name" value="main_package" />
-    <!-- SHARED -->
     <xacro:include filename="$(find ${package_name})/description/shared/inertial_macros.xacro" />
     <xacro:include filename="$(find ${package_name})/description/shared/materials.xacro" />
     <xacro:include filename="$(find ${package_name})/description/shared/properties.xacro" />
     <xacro:include filename="$(find ${package_name})/description/shared/supports.urdf.xacro" />
-    <!-- FUNCTIONAL -->
     <xacro:include filename="$(find ${package_name})/description/functional/depth_camera.urdf.xacro" />
     <xacro:include filename="$(find ${package_name})/description/functional/display.urdf.xacro" />
@@ -16,13 +14,10 @@
     <xacro:include filename="$(find ${package_name})/description/functional/stop_button.urdf.xacro" />
     <xacro:include filename="$(find ${package_name})/description/functional/wheel/wheel_100mm_light.urdf.xacro" />
-    <!-- ROBOT -->
     <xacro:include filename="$(find ${package_name})/description/robot/robot_core.xacro" />
     <xacro:include filename="$(find ${package_name})/description/robot/robot_level_1.xacro" />
     <xacro:include filename="$(find ${package_name})/description/robot/robot_level_2.xacro" />
     <xacro:include filename="$(find ${package_name})/description/robot/robot_level_3.xacro" />
-    <!-- GAZEBO -->
     <xacro:include filename="$(find ${package_name})/description/gazebo/robot_gazebo.gazebo.xacro" />
     <xacro:robot_gazebo prefix="" />
-    <!-- ROS2 CONTROL -->
     <xacro:include filename="$(find ${package_name})/description/ros2_control/robot_ros2.ros2_control.xacro" />
     <xacro:robot_ros2_control name="robot" use_sim="$(arg use_sim)" />

File: src/main_package/description/robot/robot_core.xacro (robot description, xacro)
@@ -1,7 +1,5 @@
 <?xml version="1.0"?>
 <robot xmlns:xacro="http://www.ros.org/wiki/xacro">
-    <!-- BASE LINK -->
     <link name="base_link"></link>
-    <!-- CHASSIS LINK -->
     <joint name="chassis_joint" type="fixed">
         <parent link="base_link" />
@@ -31,149 +29,24 @@
         <material>Gazebo/White</material>
     </gazebo>
-    <!-- WHEELS -->
-    <!-- left wheel -->
-    <!-- Wheel1 -->
     <xacro:omni_wheel prefix="wheel1" parent="base_link">
         <origin
             xyz="-${chassis_inner_length/2 + wheel_thickness/2} ${chassis_inner_width/2 + wheel_thickness/2} ${wheel_radius/2}"
             rpy="0 ${pi/2} ${pi*3/4}" />
-        <!-- <origin xyz="-0.35 0.35 0.05" rpy="0 ${pi/2} ${pi*3/4}" /> -->
     </xacro:omni_wheel>
-    <!-- <joint name="left_wheel_joint" type="continuous">
-        <parent link="base_link" />
-        <child link="left_wheel" />
-        <origin
-            xyz="-${chassis_inner_length/2 + wheel_thickness/2} ${chassis_inner_width/2 + wheel_thickness/2} ${wheel_radius/2}"
-            rpy="-${pi/2} 0 0.785" />
-        <axis xyz="0 0 -1" />
-    </joint>
-    <link name="left_wheel">
-        <visual>
-            <geometry>
-                <cylinder radius="${wheel_radius}" length="${wheel_thickness}" />
-            </geometry>
-            <material name="blue" />
-        </visual>
-        <collision>
-            <geometry>
-                <sphere radius="${wheel_radius}" />
-            </geometry>
-        </collision>
-        <xacro:inertial_cylinder
-            mass="1.0" length="${wheel_thickness}" radius="${wheel_radius}">
-            <origin xyz="0 0 0" rpy="0 0 0" />
-        </xacro:inertial_cylinder>
-    </link>
-    <gazebo reference="left_wheel">
-        <material>Gazebo/Blue</material>
-    </gazebo> -->
-    <!-- front wheel -->
-    <!-- Wheel0 -->
     <xacro:omni_wheel prefix="wheel0" parent="base_link">
         <origin
             xyz="${chassis_inner_length/2 + wheel_thickness/2} ${chassis_inner_width/2 + wheel_thickness/2} ${wheel_radius/2}"
             rpy="0 ${pi/2} ${pi/4}" />
-        <!-- <origin xyz="0.35 0.35 0.05" rpy="0 ${pi/2} ${pi/4}" /> -->
     </xacro:omni_wheel>
-    <!-- <joint name="front_wheel_joint" type="continuous">
-        <parent link="base_link" />
-        <child link="front_wheel" />
-        <origin
-            xyz="${chassis_inner_length/2 + wheel_thickness/2} ${chassis_inner_width/2 + wheel_thickness/2} ${wheel_radius/2}"
-            rpy="-${pi/2} 0 -0.785" />
-        <axis xyz="0 0 -1" />
-    </joint>
-    <link name="front_wheel">
-        <visual>
-            <geometry>
-                <cylinder radius="${wheel_radius}" length="${wheel_thickness}" />
-            </geometry>
-            <material name="blue" />
-        </visual>
-        <collision>
-            <geometry>
-                <sphere radius="${wheel_radius}" />
-            </geometry>
-        </collision>
-        <xacro:inertial_cylinder mass="1.0" length="${wheel_thickness}" radius="${wheel_radius}">
-            <origin xyz="0 0 0" rpy="0 0 0" />
-        </xacro:inertial_cylinder>
-    </link>
-    <gazebo reference="front_wheel">
-        <material>Gazebo/Blue</material>
-    </gazebo> -->
-    <!-- right wheel -->
-    <!-- Wheel3 -->
     <xacro:omni_wheel prefix="wheel3" parent="base_link">
         <origin
             xyz="-${chassis_inner_length/2 + wheel_thickness/2} -${chassis_inner_width/2 + wheel_thickness/2} ${wheel_radius/2}"
             rpy="0 ${pi/2} ${-pi*3/4}" />
-        <!-- <origin xyz="-0.35 -0.35 0.05" rpy="0 ${pi/2} ${-pi*3/4}" /> -->
     </xacro:omni_wheel>
-    <!-- <joint name="right_wheel_joint" type="continuous">
-        <parent link="base_link" />
-        <child link="right_wheel" />
-        <origin
-            xyz="${chassis_inner_length/2 + wheel_thickness/2} -${chassis_inner_width/2 + wheel_thickness/2} ${wheel_radius/2}"
-            rpy="${pi/2} ${pi} 0.785" />
-        <axis xyz="0 0 -1" />
-    </joint>
-    <link name="right_wheel">
-        <visual>
-            <geometry>
-                <cylinder radius="${wheel_radius}" length="${wheel_thickness}" />
-            </geometry>
-            <material name="blue" />
-        </visual>
-        <collision>
-            <geometry>
-                <sphere radius="${wheel_radius}" />
-            </geometry>
-        </collision>
-        <xacro:inertial_cylinder mass="1.0" length="${wheel_thickness}" radius="${wheel_radius}">
-            <origin xyz="0 0 0" rpy="0 0 0" />
-        </xacro:inertial_cylinder>
-    </link>
-    <gazebo reference="right_wheel">
-        <material>Gazebo/Blue</material>
-    </gazebo> -->
-    <!-- back wheel -->
-    <!-- Wheel2 -->
     <xacro:omni_wheel prefix="wheel2" parent="base_link">
         <origin
             xyz="${chassis_inner_length/2 + wheel_thickness/2} -${chassis_inner_width/2 + wheel_thickness/2} ${wheel_radius/2}"
             rpy="0 ${pi/2} ${-pi/4}" />
-        <!-- <origin xyz="0.35 -0.35 0.05" rpy="0 ${pi/2} ${-pi/4}" /> -->
     </xacro:omni_wheel>
-    <!-- <joint name="back_wheel_joint" type="continuous">
-        <parent link="base_link" />
-        <child link="back_wheel" />
-        <origin
-            xyz="-${chassis_inner_length/2 + wheel_thickness/2} -${chassis_inner_width/2 + wheel_thickness/2} ${wheel_radius/2}"
-            rpy="${pi/2} ${pi} -0.785" />
-        <axis xyz="0 0 -1" />
-    </joint>
-    <link name="back_wheel">
-        <visual>
-            <geometry>
-                <cylinder radius="${wheel_radius}" length="${wheel_thickness}" />
-            </geometry>
-            <material name="blue" />
-        </visual>
-        <collision>
-            <geometry>
-                <sphere radius="${wheel_radius}" />
-            </geometry>
-        </collision>
-        <xacro:inertial_cylinder mass="1.0" length="${wheel_thickness}" radius="${wheel_radius}">
-            <origin xyz="0 0 0" rpy="0 0 0" />
-        </xacro:inertial_cylinder>
-    </link>
-    <gazebo reference="back_wheel">
-        <material>Gazebo/Blue</material>
-    </gazebo> -->
-    <!-- FRAME -->
-    <!-- CORNERS -->
-    <!-- left corner -->
     <xacro:corner_frame nameprefix="frame_left_corner_top" parent="base_link" bx="${chassis_outer_corner}"
         by="${chassis_outer_thickness}"
@@ -189,5 +62,4 @@
             rpy="0 0 0.785" />
     </xacro:corner_frame>
-    <!-- front corner -->
     <xacro:corner_frame nameprefix="frame_front_corner_top" parent="base_link" bx="${chassis_outer_corner}"
         by="${chassis_outer_thickness}"
@@ -203,5 +75,4 @@
             rpy="0 0 -0.785" />
     </xacro:corner_frame>
-    <!-- right corner -->
     <xacro:corner_frame nameprefix="frame_right_corner_top" parent="base_link" bx="${chassis_outer_corner}"
         by="${chassis_outer_thickness}"
@@ -217,5 +88,4 @@
             rpy="0 0 0.785" />
     </xacro:corner_frame>
-    <!-- back corner -->
     <xacro:corner_frame nameprefix="frame_back_corner_top" parent="base_link" bx="${chassis_outer_corner}"
         by="${chassis_outer_thickness}"
@@ -231,6 +101,4 @@
             rpy="0 0 -0.785" />
     </xacro:corner_frame>
-    <!-- SIDES -->
-    <!-- left-front side -->
     <xacro:side_frame nameprefix="frame_left_front_side_top" bx="${chassis_outer_side}" by="${chassis_outer_thickness}"
         bz="${chassis_outer_thickness}">
@@ -244,5 +112,4 @@
             rpy="0 0 0" />
     </xacro:side_frame>
-    <!-- front-right side -->
     <xacro:side_frame nameprefix="frame_front_right_side_top" bx="${chassis_outer_thickness}" by="${chassis_outer_side}"
         bz="${chassis_outer_thickness}">
@@ -256,5 +123,4 @@
             rpy="0 0 0" />
     </xacro:side_frame>
-    <!-- right-back side -->
     <xacro:side_frame nameprefix="frame_right_back_side_top" bx="${chassis_outer_side}" by="${chassis_outer_thickness}"
         bz="${chassis_outer_thickness}">
@@ -268,5 +134,4 @@
             rpy="0 0 0" />
     </xacro:side_frame>
-    <!-- back-left side -->
     <xacro:side_frame nameprefix="frame_back_left_side_top" bx="${chassis_outer_thickness}" by="${chassis_outer_side}"
         bz="${chassis_outer_thickness}">

File: src/main_package/description/robot/robot_level_1.xacro (robot description, xacro)
@@ -1,5 +1,4 @@
 <?xml version="1.0"?>
 <robot xmlns:xacro="http://www.ros.org/wiki/xacro">
-    <!-- LEVEL 1 CENTER -->
     <joint name="level_1_center_joint" type="fixed">
         <parent link="base_link" />
@@ -9,18 +8,6 @@
             ryp="0 0 0" />
     </joint>
-    <!-- <link name="level_1_center_link">
-        <visual>
-            <geometry>
-                <box size="${level_1_base_length} ${level_1_base_width} 0.1" />
-            </geometry>
-            <material name="red" />
-        </visual>
-    </link>
-    <gazebo reference="level_1_center_link">
-        <material>Gazebo/Red</material>
-    </gazebo> -->
     <link name="level_1_center_link">
     </link>
-    <!-- LIDAR -->
     <xacro:lidar nameprefix="laser"
         parent="level_1_center_link"
@@ -31,5 +18,4 @@
         <frame_name>laser_frame</frame_name>
     </xacro:lidar>
-    <!-- BASE PLATE -->
     <xacro:base_plate nameprefix="level_1_base_plate_x"
         parent="level_1_center_link"
@@ -48,6 +34,4 @@
             rpy="0 0 0" />
     </xacro:base_plate>
-    <!-- CORNER -->
-    <!-- left corner -->
     <xacro:corner_frame nameprefix="l1_frame_left_corner"
         parent="level_1_center_link"
@@ -59,5 +43,4 @@
             rpy="0 0 0.785" />
     </xacro:corner_frame>
-    <!-- front corner -->
     <xacro:corner_frame nameprefix="l1_frame_front_corner"
         parent="level_1_center_link"
@@ -69,5 +52,4 @@
             rpy="0 0 -0.785" />
     </xacro:corner_frame>
-    <!-- right corner -->
     <xacro:corner_frame nameprefix="l1_frame_right_corner"
         parent="level_1_center_link"
@@ -79,5 +61,4 @@
             rpy="0 0 0.785" />
     </xacro:corner_frame>
-    <!-- back corner -->
     <xacro:corner_frame nameprefix="l1_frame_back_corner"
         parent="level_1_center_link"
@@ -89,5 +70,4 @@
             rpy="0 0 -0.785" />
     </xacro:corner_frame>
-    <!-- SUPPORT -->
     <xacro:support_cylinder nameprefix="l1_front_left_support_cylinder"
         parent="level_2_center_link"

File: src/main_package/description/robot/robot_level_2.xacro (robot description, xacro)
@@ -1,5 +1,4 @@
 <?xml version="1.0"?>
 <robot xmlns:xacro="http://www.ros.org/wiki/xacro">
-    <!-- LEVEL 2 CENTER -->
     <joint name="level_2_center_joint" type="fixed">
         <parent link="base_link" />
@@ -9,19 +8,6 @@
             ryp="0 0 0" />
     </joint>
-    <!-- <link name="level_2_center_link">
-        <visual>
-            <geometry>
-                <box size="${level_2_base_length} ${level_2_base_width} 0.1" />
-            </geometry>
-            <material name="red" />
-        </visual>
-    </link>
-    <gazebo reference="level_2_center_link">
-        <material>Gazebo/Red</material>
-    </gazebo> -->
     <link name="level_2_center_link">
     </link>
-    <!-- ARM -->
-    <!-- CPU -->
     <joint name="$cpu_joint" type="fixed">
         <parent link="level_2_center_link" />
@@ -51,5 +37,4 @@
         <material>Gazebo/Green</material>
     </gazebo>
-    <!-- NETWORK INTERFACE -->
     <joint name="$network_joint" type="fixed">
         <parent link="level_2_center_link" />
@@ -79,5 +64,4 @@
         <material>Gazebo/Green</material>
     </gazebo>
-    <!-- BASE PLATE -->
     <xacro:base_plate nameprefix="level_2_base_plate_x"
         parent="level_2_center_link"
@@ -96,6 +80,4 @@
             rpy="0 0 0" />
     </xacro:base_plate>
-    <!-- CORNER -->
-    <!-- left corner -->
     <xacro:corner_frame nameprefix="l2_frame_left_corner"
         parent="level_2_center_link"
@@ -107,5 +89,4 @@
             rpy="0 0 0.785" />
     </xacro:corner_frame>
-    <!-- front corner -->
     <xacro:corner_frame nameprefix="l2_frame_front_corner"
         parent="level_2_center_link"
@@ -117,5 +98,4 @@
             rpy="0 0 -0.785" />
     </xacro:corner_frame>
-    <!-- right corner -->
     <xacro:corner_frame nameprefix="l2_frame_right_corner"
         parent="level_2_center_link"
@@ -127,5 +107,4 @@
             rpy="0 0 0.785" />
     </xacro:corner_frame>
-    <!-- back corner -->
     <xacro:corner_frame nameprefix="l2_frame_back_corner"
         parent="level_2_center_link"
@@ -137,5 +116,4 @@
             rpy="0 0 -0.785" />
     </xacro:corner_frame>
-    <!-- SUPPORT -->
     <xacro:support_cylinder nameprefix="l2_front_left_support_cylinder"
         parent="level_3_center_link"

File: src/main_package/description/robot/robot_level_3.xacro (robot description, xacro)
@@ -1,5 +1,4 @@
 <?xml version="1.0"?>
 <robot xmlns:xacro="http://www.ros.org/wiki/xacro">
-    <!-- LEVEL 3 CENTER -->
     <joint name="level_3_center_joint" type="fixed">
         <parent link="base_link" />
@@ -9,18 +8,6 @@
             ryp="0 0 0" />
     </joint>
-    <!-- <link name="level_3_center_link">
-        <visual>
-            <geometry>
-                <box size="${level_3_base_length} ${level_3_base_width} 0.1" />
-            </geometry>
-            <material name="red" />
-        </visual>
-    </link>
-    <gazebo reference="level_3_center_link">
-        <material>Gazebo/Red</material>
-    </gazebo> -->
     <link name="level_3_center_link">
     </link>
-    <!-- DISPLAY -->
     <joint name="display_camera_top_joint" type="fixed">
         <parent link="level_3_center_link" />
@@ -37,5 +24,4 @@
         <origin xyz="${display_support_radius + display_length/2} 0 -${display_height/2}" rpy="0 0 0" />
     </xacro:display>
-    <!-- DISPLAY SUPPORT -->
     <xacro:support_cylinder nameprefix="l3_left_support_cylinder"
         parent="level_3_center_link"
@@ -56,5 +42,4 @@
         <origin xyz="${display_offset_x} -${display_offset_y} ${display_support_height/2}" rpy="0 0 0" />
     </xacro:support_cylinder>
-    <!-- CAMERA -->
     <xacro:depth_camera nameprefix="camera_1"
         parent="display_camera_top_link"
@@ -78,5 +63,4 @@
             rpy="0 0 0" />
     </xacro:depth_camera>
-    <!-- MIC -->
     <xacro:mic nameprefix="mic"
         parent="level_3_center_link"
@@ -90,5 +74,4 @@
         <origin xyz="${mic_offset_x} -${mic_offset_y} ${mic_base_length/2}" rpy="0 0 0" />
     </xacro:mic>
-    <!-- STOP BUTTON -->
     <xacro:stop_button nameprefix="stop_button"
         parent="level_3_center_link"
@@ -99,5 +82,4 @@
             rpy="0 0 0" />
     </xacro:stop_button>
-    <!-- BASE PLATE -->
     <xacro:base_plate nameprefix="level_3_base_plate"
         parent="level_3_center_link"

File: src/main_package/description/ros2_control/robot_ros2.ros2_control.xacro (robot description, xacro)
@@ -11,6 +11,5 @@
         </xacro:if>
         <xacro:if value="${use_sim}">
-          <!-- <plugin>gz_ros2_control/GazeboSimSystem</plugin> -->
-          <plugin>ign_ros2_control/IgnitionSystem</plugin>
+          <plugin>gazebo_ros2_control/GazeboSystem</plugin>
         </xacro:if>
       </hardware>
