Commit message: model showing  need to fix speed issues

File: src/main_package/description/shared/inertial_macros.xacro (robot description, xacro)
@@ -1,7 +1,4 @@
 <?xml version="1.0"?>
 <robot xmlns:xacro="http://www.ros.org/wiki/xacro">
-    <!-- Specify some standard inertial calculations
-    https://en.wikipedia.org/wiki/List_of_moments_of_inertia -->
-    <!-- These make use of xacro's mathematical functionality -->
     <xacro:macro name="inertial_cylinder" params="mass length radius *origin">
         <inertial>

File: src/main_package/description/shared/materials.xacro (robot description, xacro)
@@ -1,37 +1,28 @@
 <?xml version="1.0"?>
 <robot xmlns:xacro="http://www.ros.org/wiki/xacro">
-    <!-- DISPLAY -->
     <material name="black">
         <color rgba="0 0 0 1" />
     </material>
-    <!-- SUPPORT -->
     <material name="grey">
         <color rgba="0.5 0.5 0.5 1" />
     </material>
-    <!-- MIC -->
     <material name="dark_grey">
         <color rgba="0.25 0.25 0.25 1" />
     </material>
-    <!-- MIC -->
     <material name="orange">
         <color rgba="1 0.3 0.1 1" />
     </material>
-    <!-- FRAME -->
     <material name="white">
         <color rgba="1 1 1 1" />
     </material>
-    <!-- BASE PLATE -->
     <material name="white_transparent">
         <color rgba="1 1 1 0.5" />
     </material>
-    <!-- STOP BUTTON -->
     <material name="red">
         <color rgba="1 0 0 1" />
     </material>
-    <!-- CPU -->
     <material name="green">
         <color rgba="0.2 1 0.2 1" />
     </material>
-    <!-- WHEEL -->
     <material name="blue">
         <color rgba="0.2 0.2 1 1" />
@@ -40,9 +31,7 @@
         <color rgba="0.6 0.6 0.6 1" />
     </material>
-    <!-- CAMERA -->
     <material name="yellow">
         <color rgba="1 1 0.6 1" />
     </material>
-    <!-- LIDAR -->
     <material name="purple">
         <color rgba="0.627 0.125 0.941 1" />

File: src/main_package/description/shared/properties.xacro (robot description, xacro)
@@ -1,21 +1,9 @@
 <?xml version="1.0"?>
 <robot xmlns:xacro="http://www.ros.org/wiki/xacro">
-    <!--
-        LENGTH: x
-        WIDTH: y
-        HEIGHT: z
-    -->
-    <!-- ROBOT CORE PROPERTIES -->
     <xacro:property name="metal_thickness" value="0.003" />
     <xacro:property name="metal_density" value="7850.0" />
-    <!--
-    mass = width * height * metal_thickness * metal_density
-    mass = length * height * metal_thickness * metal_density
-    -->
-    <!-- WHEEL PROPS -->
     <xacro:property name="wheel_radius" value="0.050" />
     <xacro:property name="wheel_thickness" value="0.038" />
     <xacro:property name="wheel_padding" value="0.005" />
-    <!-- CHASSIS & FRAME PROPS -->
     <xacro:property name="chassis_length" value="0.500" />
     <xacro:property name="chassis_width" value="0.500" />
@@ -30,5 +18,4 @@
     <xacro:property name="chassis_empty_space_length" value="${(chassis_length - chassis_outer_thickness*4)/3}" />
     <xacro:property name="chassis_empty_space_width" value="${(chassis_width - chassis_outer_thickness*4)/3}" />
-    <!-- ROBOT LEVEL 1 PROPERTIES -->
     <xacro:property name="level_1_height_displacement" value="${chassis_clearance + chassis_height}" />
     <xacro:property name="level_1_length_displacement" value="0.000" />
@@ -50,9 +37,7 @@
     <xacro:property name="level_1_center_z"
         value="${level_1_height_displacement + metal_thickness}" />
-    <!-- LIDAR -->
     <xacro:property name="lidar_radius" value="0.030" />
     <xacro:property name="lidar_length" value="0.068" />
     <xacro:property name="lidar_weight" value="0.400" />
-    <!-- ROBOT LEVEL 2 PROPERTIES -->
     <xacro:property name="level_2_height_displacement"
         value="${level_1_height_displacement + metal_thickness + level_1_support_height}" />
@@ -77,5 +62,4 @@
     <xacro:property name="level_2_center_z"
         value="${level_2_height_displacement + metal_thickness}" />
-    <!-- CPU -->
     <xacro:property name="cpu_length" value="0.105" />
     <xacro:property name="cpu_width" value="0.145" />
@@ -84,5 +68,4 @@
     <xacro:property name="cpu_offset_x" value="-0.070" />
     <xacro:property name="cpu_offset_y" value="-0.090" />
-    <!-- NETWORK INTERFACE -->
     <xacro:property name="network_length" value="0.150" />
     <xacro:property name="network_width" value="0.060" />
@@ -91,5 +74,4 @@
     <xacro:property name="network_offset_x" value="-0.070" />
     <xacro:property name="network_offset_y" value="0.040" />
-    <!-- ROBOT LEVEL 3 PROPERTIES -->
     <xacro:property name="level_3_height_displacement"
         value="${level_2_height_displacement + metal_thickness + level_2_support_height}" />
@@ -108,7 +90,4 @@
     <xacro:property name="level_3_center_z"
         value="${level_3_height_displacement + metal_thickness}" />
-    <!-- DEPTH CAMERA -->
-    <!-- NAME | x y z | weight | fixture_radius fixture_length -->
-    <!-- intel REALSENSE | 0.026 0.124 0.029 | 0.38 | 0.0125 0.073 -->
     <xacro:property name="intel_camera_length" value="0.026" />
     <xacro:property name="intel_camera_width" value="0.124" />
@@ -117,5 +96,4 @@
     <xacro:property name="intel_camera_fixture_radius" value="0.0125" />
     <xacro:property name="intel_camera_fixture_length" value="0.073" />
-    <!-- DISPLAY -->
     <xacro:property name="display_length" value="0.015" />
     <xacro:property name="display_width" value="0.235" />
@@ -126,5 +104,4 @@
     <xacro:property name="display_offset_x" value="-0.100" />
     <xacro:property name="display_offset_y" value="0.055" />
-    <!-- MIC -->
     <xacro:property name="mic_base_length" value="0.010" />
     <xacro:property name="mic_base_radius" value="0.036" />
@@ -136,5 +113,4 @@
     <xacro:property name="mic_offset_x" value="0.030" />
     <xacro:property name="mic_offset_y" value="0.070" />
-    <!-- STOP BUTTON -->
     <xacro:property name="stop_button_radius" value="0.018" />
     <xacro:property name="stop_button_length" value="0.030" />

File: src/main_package/description/shared/supports.urdf.xacro (robot description, xacro)
@@ -1,5 +1,4 @@
 <?xml version="1.0"?>
 <robot xmlns:xacro="http://www.ros.org/wiki/xacro">
-    <!-- BASE CORNER -->
     <xacro:macro name="corner_frame" params="nameprefix parent bx by bz *origin">
         <joint name="${nameprefix}_joint" type="fixed">
@@ -31,5 +30,4 @@
         </gazebo>
     </xacro:macro>
-    <!-- BASE SIDE -->
     <xacro:macro name="side_frame" params="nameprefix bx by bz *origin">
         <joint name="${nameprefix}_joint" type="fixed">
@@ -61,5 +59,4 @@
         </gazebo>
     </xacro:macro>
-    <!-- SUPPORT CYLINDER -->
     <xacro:macro name="support_cylinder" params="nameprefix parent length radius *origin">
         <joint name="${nameprefix}_joint" type="fixed">
@@ -90,5 +87,4 @@
         </gazebo>
     </xacro:macro>
-    <!-- BASE PLATE -->
     <xacro:macro name="base_plate" params="nameprefix parent bx by bz *origin">
         <joint name="${nameprefix}_joint" type="fixed">
