Commit message: omni wheel but different gazebo version

File: src/main_package/description/functional/lidar.urdf.xacro (robot description, xacro)
@@ -48,5 +48,5 @@
                 <plugin name="${nameprefix}_controller" filename="libgazebo_ros_ray_sensor.so">
                     <ros>
-                        <argument>~/out:=scan</argument>
+                        <argument>--ros-args --remap ~/out:=scan</argument>
                     </ros>
                     <output_type>sensor_msgs/LaserScan</output_type>

File: src/main_package/description/robot/robot.urdf.xacro (robot description, xacro)
@@ -1,4 +1,6 @@
 <?xml version="1.0"?>
 <robot xmlns:xacro="http://www.ros.org/wiki/xacro" name="robot">
+    <xacro:arg name="prefix" default="" />
+    <xacro:arg name="use_sim" default="false" />
     <xacro:property name="package_name" value="main_package" />
     <!-- SHARED -->
@@ -13,4 +15,5 @@
     <xacro:include filename="$(find ${package_name})/description/functional/mic.urdf.xacro" />
     <xacro:include filename="$(find ${package_name})/description/functional/stop_button.urdf.xacro" />
+    <xacro:include filename="$(find ${package_name})/description/functional/wheel/wheel_100mm_light.urdf.xacro" />
     <!-- ROBOT -->
     <xacro:include filename="$(find ${package_name})/description/robot/robot_core.xacro" />
@@ -18,3 +21,9 @@
     <xacro:include filename="$(find ${package_name})/description/robot/robot_level_2.xacro" />
     <xacro:include filename="$(find ${package_name})/description/robot/robot_level_3.xacro" />
+    <!-- GAZEBO -->
+    <xacro:include filename="$(find ${package_name})/description/gazebo/robot_gazebo.gazebo.xacro" />
+    <xacro:robot_gazebo prefix="" />
+    <!-- ROS2 CONTROL -->
+    <xacro:include filename="$(find ${package_name})/description/ros2_control/robot_ros2.ros2_control.xacro" />
+    <xacro:robot_ros2_control name="robot" use_sim="$(arg use_sim)" />
 </robot>

File: src/main_package/description/robot/robot_core.xacro (robot description, xacro)
@@ -1,7 +1,4 @@
 <?xml version="1.0"?>
 <robot xmlns:xacro="http://www.ros.org/wiki/xacro">
-    <!-- WHEEL PROPS -->
-    <xacro:property name="wheel_radius" value="0.050" />
-    <xacro:property name="wheel_thickness" value="0.038" />
     <!-- BASE LINK -->
     <link name="base_link"></link>
@@ -36,5 +33,11 @@
     <!-- WHEELS -->
     <!-- left wheel -->
-    <joint name="left_wheel_joint" type="continuous">
+    <!-- Wheel1 -->
+    <xacro:omni_wheel prefix="wheel1" parent="base_link">
+        <origin
+            xyz="-${chassis_inner_length/2 + wheel_thickness/2} ${chassis_inner_width/2 + wheel_thickness/2} ${wheel_radius/2}"
+            rpy="0 ${pi/2} ${pi*3/4}" />
+    </xacro:omni_wheel>
+    <!-- <joint name="left_wheel_joint" type="continuous">
         <parent link="base_link" />
         <child link="left_wheel" />
@@ -63,7 +66,13 @@
     <gazebo reference="left_wheel">
         <material>Gazebo/Blue</material>
-    </gazebo>
+    </gazebo> -->
     <!-- front wheel -->
-    <joint name="front_wheel_joint" type="continuous">
+    <!-- Wheel0 -->
+    <xacro:omni_wheel prefix="wheel0" parent="base_link">
+        <origin
+            xyz="${chassis_inner_length/2 + wheel_thickness/2} ${chassis_inner_width/2 + wheel_thickness/2} ${wheel_radius/2}"
+            rpy="0 ${pi/2} ${pi/4}" />
+    </xacro:omni_wheel>
+    <!-- <joint name="front_wheel_joint" type="continuous">
         <parent link="base_link" />
         <child link="front_wheel" />
@@ -91,7 +100,13 @@
     <gazebo reference="front_wheel">
         <material>Gazebo/Blue</material>
-    </gazebo>
+    </gazebo> -->
     <!-- right wheel -->
-    <joint name="right_wheel_joint" type="continuous">
+    <!-- Wheel3 -->
+    <xacro:omni_wheel prefix="wheel2" parent="base_link">
+        <origin
+            xyz="${chassis_inner_length/2 + wheel_thickness/2} -${chassis_inner_width/2 + wheel_thickness/2} ${wheel_radius/2}"
+            rpy="0 ${pi/2} ${-pi*3/4}" />
+    </xacro:omni_wheel>
+    <!-- <joint name="right_wheel_joint" type="continuous">
         <parent link="base_link" />
         <child link="right_wheel" />
@@ -119,7 +134,13 @@
     <gazebo reference="right_wheel">
         <material>Gazebo/Blue</material>
-    </gazebo>
+    </gazebo> -->
     <!-- back wheel -->
-    <joint name="back_wheel_joint" type="continuous">
+    <!-- Wheel2 -->
+    <xacro:omni_wheel prefix="wheel3" parent="base_link">
+        <origin
+            xyz="-${chassis_inner_length/2 + wheel_thickness/2} -${chassis_inner_width/2 + wheel_thickness/2} ${wheel_radius/2}"
+            rpy="0 ${pi/2} ${-pi/4}" />
+    </xacro:omni_wheel>
+    <!-- <joint name="back_wheel_joint" type="continuous">
         <parent link="base_link" />
         <child link="back_wheel" />
@@ -147,5 +168,5 @@
     <gazebo reference="back_wheel">
         <material>Gazebo/Blue</material>
-    </gazebo>
+    </gazebo> -->
     <!-- FRAME -->
     <!-- CORNERS -->

File: src/main_package/description/shared/materials.xacro (robot description, xacro)
@@ -37,4 +37,7 @@
         <color rgba="0.2 0.2 1 1" />
     </material>
+    <material name="gray">
+        <color rgba="0.6 0.6 0.6 1" />
+    </material>
     <!-- CAMERA -->
     <material name="yellow">

File: src/main_package/description/shared/properties.xacro (robot description, xacro)
@@ -13,4 +13,7 @@
     mass = length * height * metal_thickness * metal_density
     -->
+    <!-- WHEEL PROPS -->
+    <xacro:property name="wheel_radius" value="0.050" />
+    <xacro:property name="wheel_thickness" value="0.038" />
     <!-- CHASSIS & FRAME PROPS -->
     <xacro:property name="chassis_length" value="0.500" />

Commit message: balleced weight, working SLAM

File: src/main_package/description/functional/lidar.urdf.xacro (robot description, xacro)
@@ -29,5 +29,5 @@
             <sensor name="${nameprefix}" type="ray">
                 <pose> 0 0 0 0 0 0 </pose>
-                <visualize>true</visualize>
+                <visualize>false</visualize>
                 <update_rate>10</update_rate>
                 <ray>

File: src/main_package/description/functional/wheel/wheel_100mm.urdf.xacro (robot description, xacro)
@@ -23,5 +23,5 @@
       <inertial>
         <mass value="0.002" />
-        <inertia ixx="0.000001" ixy="0" ixz="0" iyy="0.000001" iyz="0" izz="0.000001" />
+        <inertia ixx="0.00001" ixy="0" ixz="0" iyy="0.00001" iyz="0" izz="0.00001" />
       </inertial>
     </link>
@@ -50,5 +50,5 @@
       <xacro:insert_block name="joint_origin" />
       <axis xyz="0 0 1" />
-      <dynamics damping="1.0" />
+      <dynamics damping="0.7" />
     </joint>
     <transmission name="${prefix}_shaft_trans">
@@ -71,10 +71,9 @@
       </visual>
       <inertial>
-        <mass value="0.025" />
-        <inertia ixx="0.0001" ixy="0" ixz="0" iyy="0.0001" iyz="0" izz="0.0001" />
+        <mass value="0.25" />
+        <inertia ixx="0.00235" ixy="0" ixz="0" iyy="0.00235" iyz="0" izz="0.00004" />
       </inertial>
     </link>
     <gazebo reference="${prefix}_housing_link">
-      <selfCollide>false</selfCollide>
       <material>Gazebo/Gray</material>
       <mu1>0.8</mu1>

File: src/main_package/description/functional/wheel/wheel_100mm_light.urdf.xacro (robot description, xacro)
@@ -1,9 +1,9 @@
 <?xml version="1.0"?>
 <robot xmlns:xacro="http://ros.org/wiki/xacro">
-  <xacro:macro name="omni_wheel" params="prefix parent *joint_origin">
+  <xacro:macro name="omni_wheel" params="prefix parent *origin">
     <joint name="${prefix}_shaft_joint" type="continuous">
       <parent link="${parent}" />
       <child link="${prefix}_housing_link" />
-      <xacro:insert_block name="joint_origin" />
+      <xacro:insert_block name="origin" />
       <axis xyz="0 0 1" />
       <dynamics damping="0.7" />
@@ -22,5 +22,5 @@
       <visual>
         <geometry>
-          <cylinder length="0.040" radius="0.05" />
+          <cylinder length="0.040" radius="0.0675" />
         </geometry>
         <origin xyz="0 0 0" rpy="0 0 0" />
@@ -29,5 +29,5 @@
       <collision>
         <geometry>
-          <cylinder length="0.040" radius="0.05" />
+          <sphere radius="0.0675" />
         </geometry>
         <origin xyz="0 0 0" rpy="0 0 0" />
@@ -35,16 +35,10 @@
       </collision>
       <inertial>
-        <mass value="1.288" />
-        <inertia ixx="0.00235" ixy="0" ixz="0" iyy="0.00235" iyz="0" izz="0.00004" />
+        <mass value="0.25" />
+        <inertia ixx="0.00235" ixy="0" ixz="0" iyy="0.00235" iyz="0" izz="0.015" />
       </inertial>
     </link>
     <gazebo reference="${prefix}_housing_link">
-      <selfCollide>false</selfCollide>
       <material>Gazebo/Gray</material>
-      <mu1>0.8</mu1>
-      <mu2>0.05</mu2>
-      <fdir1>0 1.0 0</fdir1>
-      <kp value="3000.0" />
-      <kd value="3000.0" />
     </gazebo>
   </xacro:macro>

File: src/main_package/description/robot/robot.urdf.xacro (robot description, xacro)
@@ -10,8 +10,9 @@
     <xacro:include filename="$(find ${package_name})/description/functional/depth_camera.urdf.xacro" />
     <xacro:include filename="$(find ${package_name})/description/functional/display.urdf.xacro" />
+    <xacro:include filename="$(find ${package_name})/description/functional/arm/temparm.xacro" />
     <xacro:include filename="$(find ${package_name})/description/functional/lidar.urdf.xacro" />
     <xacro:include filename="$(find ${package_name})/description/functional/mic.urdf.xacro" />
     <xacro:include filename="$(find ${package_name})/description/functional/stop_button.urdf.xacro" />
-    <xacro:include filename="$(find ${package_name})/description/functional/wheel/wheel_100mm.urdf.xacro" />
+    <xacro:include filename="$(find ${package_name})/description/functional/wheel/wheel_100mm_light.urdf.xacro" />
     <xacro:include filename="$(find ${package_name})/description/robot/robot_core.xacro" />
     <xacro:include filename="$(find ${package_name})/description/robot/robot_level_1.xacro" />

File: src/main_package/description/robot/robot_core.xacro (robot description, xacro)
@@ -36,20 +36,20 @@
         <material>Gazebo/White</material>
     </gazebo>
-    <xacro:omni_wheel prefix="wheel3" parent="base_link">
+    <xacro:omni_wheel prefix="wheel1" parent="base_link">
         <origin
             xyz="-${chassis_inner_length/2 + wheel_thickness/2} ${chassis_inner_width/2 + wheel_thickness/2} ${wheel_radius/2}"
             rpy="0 ${pi/2} ${pi*3/4}" />
     </xacro:omni_wheel>
-    <xacro:omni_wheel prefix="wheel2" parent="base_link">
+    <xacro:omni_wheel prefix="wheel0" parent="base_link">
         <origin
             xyz="${chassis_inner_length/2 + wheel_thickness/2} ${chassis_inner_width/2 + wheel_thickness/2} ${wheel_radius/2}"
             rpy="0 ${pi/2} ${pi/4}" />
     </xacro:omni_wheel>
-    <xacro:omni_wheel prefix="wheel1" parent="base_link">
+    <xacro:omni_wheel prefix="wheel3" parent="base_link">
         <origin
             xyz="-${chassis_inner_length/2 + wheel_thickness/2} -${chassis_inner_width/2 + wheel_thickness/2} ${wheel_radius/2}"
             rpy="0 ${pi/2} ${-pi*3/4}" />
     </xacro:omni_wheel>
-    <xacro:omni_wheel prefix="wheel0" parent="base_link">
+    <xacro:omni_wheel prefix="wheel2" parent="base_link">
         <origin
             xyz="${chassis_inner_length/2 + wheel_thickness/2} -${chassis_inner_width/2 + wheel_thickness/2} ${wheel_radius/2}"

File: src/main_package/description/robot/robot_level_2.xacro (robot description, xacro)
@@ -64,4 +64,13 @@
         <material>Gazebo/Green</material>
     </gazebo>
+    <xacro:temparm
+        nameprefix="temparm"
+        parent="level_2_center_link"
+        bx="0.05"
+        by="0.05"
+        bz="0.5"
+        mass="4.5">
+        <origin xyz="0.2 0 0.253" rpy="0 0 0" />
+    </xacro:temparm>
     <xacro:base_plate nameprefix="level_2_base_plate_x"
         parent="level_2_center_link"

File: src/main_package/description/shared/properties.xacro (robot description, xacro)
@@ -3,17 +3,17 @@
     <xacro:property name="metal_thickness" value="0.003" />
     <xacro:property name="metal_density" value="7850.0" />
-    <xacro:property name="wheel_radius" value="0.050" />
+    <xacro:property name="wheel_radius" value="0.0675" />
     <xacro:property name="wheel_thickness" value="0.04" />
     <xacro:property name="wheel_padding" value="0.005" />
     <xacro:property name="chassis_length" value="0.500" />
     <xacro:property name="chassis_width" value="0.500" />
-    <xacro:property name="chassis_inner_length" value="0.272" />
-    <xacro:property name="chassis_inner_width" value="0.272" />
+    <xacro:property name="chassis_inner_length" value="0.275" />
+    <xacro:property name="chassis_inner_width" value="0.275" />
     <xacro:property name="chassis_outer_side" value="0.272" />
-    <xacro:property name="chassis_outer_corner" value="0.162" />
+    <xacro:property name="chassis_outer_corner" value="0.160" />
     <xacro:property name="chassis_corner_margin" value="0.080" />
     <xacro:property name="chassis_outer_thickness" value="0.020" />
-    <xacro:property name="chassis_height" value="0.120" />
-    <xacro:property name="chassis_clearance" value="0.050" />
+    <xacro:property name="chassis_height" value="0.140" />
+    <xacro:property name="chassis_clearance" value="0.020" />
     <xacro:property name="chassis_empty_space_length" value="${(chassis_length - chassis_outer_thickness*4)/3}" />
     <xacro:property name="chassis_empty_space_width" value="${(chassis_width - chassis_outer_thickness*4)/3}" />
@@ -110,5 +110,5 @@
     <xacro:property name="mic_length" value="0.150" />
     <xacro:property name="mic_radius" value="0.015" />
-    <xacro:property name="mic_weight" value="0.200" />
+    <xacro:property name="mic_weight" value="0.05" />
     <xacro:property name="mic_offset_x" value="0.030" />
     <xacro:property name="mic_offset_y" value="0.070" />
