Commit message: slam

File: src/main_package/description/gazebo/robot_gazebo.gazebo.xacro (robot description, xacro)
@@ -2,10 +2,6 @@
 <robot xmlns:xacro="http://ros.org/wiki/xacro">
   <xacro:macro name="robot_gazebo" params="prefix">
-    <!-- <gazebo>
-      <plugin name="gazebo_ros2_control" filename="libgazebo_ros2_control.so">
-        <parameters>$(find main_package)/config/robot_config.yaml</parameters>
-        <parameters>$(find main_package)/params/gaz_ros2_ctl_use_sim.yaml</parameters>
-      </plugin>
-    </gazebo> -->
+    <gazebo>
+    </gazebo>
   </xacro:macro>
 </robot>

File: src/main_package/description/robot/robot_core.xacro (robot description, xacro)
@@ -2,4 +2,11 @@
 <robot xmlns:xacro="http://www.ros.org/wiki/xacro">
     <link name="base_link"></link>
+    <joint name="base_footprint_joint" type="fixed">
+        <parent link="base_link" />
+        <child link="base_footprint" />
+        <origin xyz="0 0 0" rpy="0 0 0" />
+    </joint>
+    <link name="base_footprint">
+    </link>
     <joint name="chassis_joint" type="fixed">
         <parent link="base_link" />
