Commit message: arduino python script

File: src/main_package/description/functional/wheel/wheel_100mm.urdf.xacro (robot description, xacro)
@@ -12,5 +12,5 @@
       <visual>
         <geometry>
-          <mesh filename="file://$(find main_package)description/meshes/STL/omni_barrel_100mm.stl" />
+          <mesh filename="file://$(find main_package)/description/meshes/STL/omni_barrel_100mm.stl" />
         </geometry>
         <material name="black" />
@@ -18,5 +18,5 @@
       <collision>
         <geometry>
-          <mesh filename="file://$(find main_package)description/meshes/STL/omni_barrel_100mm.stl" />
+          <mesh filename="file://$(find main_package)/description/meshes/STL/omni_barrel_100mm.stl" />
         </geometry>
       </collision>
@@ -50,5 +50,5 @@
       <xacro:insert_block name="joint_origin" />
       <axis xyz="0 0 1" />
-      <dynamics damping="0.7" />
+      <dynamics damping="1.0" />
     </joint>
     <transmission name="${prefix}_shaft_trans">
@@ -65,5 +65,5 @@
       <visual>
         <geometry>
-          <mesh filename="file://$(find main_package)description/meshes/STL/omni_housing_100mm.stl" />
+          <mesh filename="file://$(find main_package)/description/meshes/STL/omni_housing_100mm.stl" />
         </geometry>
         <origin xyz="0 0 0" rpy="0 0 0" />
@@ -76,5 +76,11 @@
     </link>
     <gazebo reference="${prefix}_housing_link">
+      <selfCollide>false</selfCollide>
       <material>Gazebo/Gray</material>
+      <mu1>0.8</mu1>
+      <mu2>0.05</mu2>
+      <fdir1>0 1.0 0</fdir1>
+      <kp value="2500.0" />
+      <kd value="2500.0" />
     </gazebo>
     <joint name="${prefix}_housing_s_joint" type="fixed">

File: src/main_package/description/functional/wheel/wheel_100mm_light.urdf.xacro (robot description, xacro)
@@ -40,10 +40,11 @@
     </link>
     <gazebo reference="${prefix}_housing_link">
+      <selfCollide>false</selfCollide>
       <material>Gazebo/Gray</material>
       <mu1>0.8</mu1>
       <mu2>0.05</mu2>
       <fdir1>0 1.0 0</fdir1>
-      <kp value="30000000.0" />
-      <kd value="50000000.0" />
+      <kp value="3000.0" />
+      <kd value="3000.0" />
     </gazebo>
   </xacro:macro>

File: src/main_package/description/robot/robot.urdf.xacro (robot description, xacro)
@@ -13,5 +13,5 @@
     <xacro:include filename="$(find ${package_name})/description/functional/mic.urdf.xacro" />
     <xacro:include filename="$(find ${package_name})/description/functional/stop_button.urdf.xacro" />
-    <xacro:include filename="$(find ${package_name})/description/functional/wheel/wheel_100mm_light.urdf.xacro" />
+    <xacro:include filename="$(find ${package_name})/description/functional/wheel/wheel_100mm.urdf.xacro" />
     <xacro:include filename="$(find ${package_name})/description/robot/robot_core.xacro" />
     <xacro:include filename="$(find ${package_name})/description/robot/robot_level_1.xacro" />

File: src/main_package/description/robot/robot_core.xacro (robot description, xacro)
@@ -36,20 +36,20 @@
         <material>Gazebo/White</material>
     </gazebo>
-    <xacro:omni_wheel prefix="wheel1" parent="base_link">
+    <xacro:omni_wheel prefix="wheel3" parent="base_link">
         <origin
             xyz="-${chassis_inner_length/2 + wheel_thickness/2} ${chassis_inner_width/2 + wheel_thickness/2} ${wheel_radius/2}"
             rpy="0 ${pi/2} ${pi*3/4}" />
     </xacro:omni_wheel>
-    <xacro:omni_wheel prefix="wheel0" parent="base_link">
+    <xacro:omni_wheel prefix="wheel2" parent="base_link">
         <origin
             xyz="${chassis_inner_length/2 + wheel_thickness/2} ${chassis_inner_width/2 + wheel_thickness/2} ${wheel_radius/2}"
             rpy="0 ${pi/2} ${pi/4}" />
     </xacro:omni_wheel>
-    <xacro:omni_wheel prefix="wheel3" parent="base_link">
+    <xacro:omni_wheel prefix="wheel1" parent="base_link">
         <origin
             xyz="-${chassis_inner_length/2 + wheel_thickness/2} -${chassis_inner_width/2 + wheel_thickness/2} ${wheel_radius/2}"
             rpy="0 ${pi/2} ${-pi*3/4}" />
     </xacro:omni_wheel>
-    <xacro:omni_wheel prefix="wheel2" parent="base_link">
+    <xacro:omni_wheel prefix="wheel0" parent="base_link">
         <origin
             xyz="${chassis_inner_length/2 + wheel_thickness/2} -${chassis_inner_width/2 + wheel_thickness/2} ${wheel_radius/2}"

File: src/main_package/description/ros2_control/robot_ros2.ros2_control.xacro (robot description, xacro)
@@ -10,4 +10,6 @@
           <param name="state_following_offset">0.0</param>
         </xacro:if>
+        <xacro:unless value="${use_sim}">
+        </xacro:unless>
         <xacro:if value="${use_sim}">
           <plugin>gazebo_ros2_control/GazeboSystem</plugin>

File: src/main_package/description/shared/properties.xacro (robot description, xacro)
@@ -4,5 +4,5 @@
     <xacro:property name="metal_density" value="7850.0" />
     <xacro:property name="wheel_radius" value="0.050" />
-    <xacro:property name="wheel_thickness" value="0.038" />
+    <xacro:property name="wheel_thickness" value="0.04" />
     <xacro:property name="wheel_padding" value="0.005" />
     <xacro:property name="chassis_length" value="0.500" />
